Commit message: Fixed imu link and added joint to joint_state_publisher

File: models/plane/plane.sdf.xacro (robot description, xacro)
@@ -63,5 +63,5 @@
       <self_collide>0</self_collide>
     </link>
-    <link name='$(arg vehicle_name)_plane/imu_link'>
+    <link name='$(arg vehicle_name)_imu_link'>
       <pose>0 0 0 0 0 0</pose>
       <inertial>
@@ -78,6 +78,6 @@
       </inertial>
     </link>
-    <joint name='plane/imu_joint' type='revolute'>
-      <child>$(arg vehicle_name)_plane/imu_link</child>
+    <joint name='$(arg vehicle_name)_imu_joint' type='revolute'>
+      <child>$(arg vehicle_name)_imu_link</child>
       <parent>$(arg vehicle_name)_base_link</parent>
       <axis>
@@ -397,5 +397,5 @@
     <plugin name='gazebo_imu_plugin' filename='libgazebo_imu_plugin.so'>
       <robotNamespace></robotNamespace>
-      <linkName>$(arg vehicle_name)_plane/imu_link</linkName>
+      <linkName>$(arg vehicle_name)_imu_link</linkName>
       <imuTopic>/imu</imuTopic>
       <gyroscopeNoiseDensity>0.0003394</gyroscopeNoiseDensity>
@@ -497,8 +497,9 @@
     <static>0</static>
     <plugin name="joint_state_publisher" filename="libgazebo_ros_joint_state_publisher.so">
-      <ros>
-        <namespace>/demo</namespace>
-        <argument>joint_states:=joint_states</argument>
-      </ros>
+      <joint_name>$(arg vehicle_name)::$(arg vehicle_name)_imu_joint</joint_name>
+      <joint_name>$(arg vehicle_name)::$(arg vehicle_name)_right_elevon_joint</joint_name>
+      <joint_name>$(arg vehicle_name)::$(arg vehicle_name)_left_elevon_joint</joint_name>
+      <joint_name>$(arg vehicle_name)::$(arg vehicle_name)_elevator_joint</joint_name>
+      <joint_name>$(arg vehicle_name)::$(arg vehicle_name)_rudder_joint</joint_name>
       <joint_name>$(arg vehicle_name)::$(arg vehicle_name)_rotor_puller_joint</joint_name>
       <update_rate>100</update_rate>

File: models/plane/plane.urdf.xacro (robot description, xacro)
@@ -36,5 +36,5 @@
       <self_collide>0</self_collide>
     </gazebo>
-    <link name='$(arg vehicle_name)_plane/imu_link'>
+    <link name='$(arg vehicle_name)_imu_link'>
       <pose rpy="0  0  0" xyz="0  0  0"/>
       <inertial>
@@ -44,7 +44,7 @@
       </inertial>
     </link>
-    <joint name="imu_joint" type="revolute">
-      <parent link="$(arg vehicle_name)_base_link"/>
-      <child link="$(arg vehicle_name)_plane/imu_link"/>
+    <joint name='$(arg vehicle_name)_imu_joint' type='revolute'>
+      <parent link="$(arg vehicle_name)_base_link"/>
+      <child link="$(arg vehicle_name)_imu_link"/>
       <origin rpy="0  0  0" xyz="0  0  0"/>
       <axis xyz="1  0  0"/>
@@ -277,5 +277,5 @@
         <plugin name='gazebo_imu_plugin' filename='libgazebo_imu_plugin.so'>
           <robotNamespace></robotNamespace>
-          <linkName>$(arg vehicle_name)_plane/imu_link</linkName>
+          <linkName>$(arg vehicle_name)_imu_link</linkName>
           <imuTopic>/imu</imuTopic>
           <gyroscopeNoiseDensity>0.0003394</gyroscopeNoiseDensity>
@@ -376,8 +376,9 @@
         </plugin>
         <plugin name="joint_state_publisher" filename="libgazebo_ros_joint_state_publisher.so">
-          <ros>
-            <namespace>/demo</namespace>
-            <argument>joint_states:=joint_states</argument>
-          </ros>
+          <joint_name>$(arg vehicle_name)::$(arg vehicle_name)_imu_joint</joint_name>
+          <joint_name>$(arg vehicle_name)::$(arg vehicle_name)_right_elevon_joint</joint_name>
+          <joint_name>$(arg vehicle_name)::$(arg vehicle_name)_left_elevon_joint</joint_name>
+          <joint_name>$(arg vehicle_name)::$(arg vehicle_name)_elevator_joint</joint_name>
+          <joint_name>$(arg vehicle_name)::$(arg vehicle_name)_rudder_joint</joint_name>
           <joint_name>$(arg vehicle_name)::$(arg vehicle_name)_rotor_puller_joint</joint_name>
           <update_rate>100</update_rate>

Commit message: added geotagged_cam in plane.sdf.xacro

File: models/plane/plane.sdf.xacro (robot description, xacro)
@@ -506,6 +506,55 @@
     </plugin>
   <xacro:if value="$(arg enable_camera)">
-    <xacro:include filename="$(arg rotors_description_dir)/geotagged_cam/geotagged_cam.sdf.xacro">
-    </xacro:include>
+    <xacro:arg name='camera_control_udp_port' default='14530' />
+      <xacro:arg name='camera_pose' default='-0.051 0 -0.162 0 0 3.14159'/>
+      <model name="geotagged_cam">
+        <link name="camera_link">
+          <inertial>
+            <!-- place holder -->
+            <pose>-0.041 0 -0.162 0 0 0</pose>
+            <mass>0.1</mass>
+            <inertia>
+              <ixx>0.001</ixx>
+              <ixy>0</ixy>
+              <ixz>0</ixz>
+              <iyy>0.001</iyy>
+              <iyz>0</iyz>
+              <izz>0.001</izz>
+            </inertia>
+          </inertial>
+          <sensor name="camera_imu" type="imu">
+            <always_on>1</always_on>
+          </sensor>
+          <sensor name="camera" type="camera">
+            <pose>$(arg camera_pose)</pose>
+            <camera>
+              <horizontal_fov>1.0</horizontal_fov>
+              <image>
+                <format>R8G8B8</format>
+                <width>640</width>
+                <height>360</height>
+              </image>
+              <clip>
+                <near>0.05</near>
+                <far>15000</far>
+              </clip>
+            </camera>
+            <always_on>1</always_on>
+            <update_rate>5</update_rate>
+            <visualize>false</visualize>
+            <plugin name="GstCameraPlugin" filename="libgazebo_gst_camera_plugin.so">
+                <robotNamespace></robotNamespace>
+                <udpPort>$(arg camera_udp_port)</udpPort>
+            </plugin>
+            <plugin name="GeotaggedImagesPlugin" filename="libgazebo_geotagged_images_plugin.so">
+              <robotNamespace></robotNamespace>
+              <interval>1</interval>
+              <width>3840</width>
+              <height>2160</height>
+              <camera_control_udp_port>$(arg camera_control_udp_port)</camera_control_udp_port>
+            </plugin>
+          </sensor>
+        </link>
+      </model>
     <joint name="geotagged_cam_joint" type="fixed">
       <parent>$(arg vehicle_name)_base_link</parent>
