Commit message: fixed typhoon legs

File: models/typhoon_h480/urdf/component_snippets.xacro (robot description, xacro)
@@ -281,5 +281,5 @@
             <joint_control_type>position_gztopic</joint_control_type>
             <gztopic>/gimbal_yaw_cmd</gztopic>
-            <joint_name>${namespace}::${namespace}_cgo3_vertical_arm_joint</joint_name>
+            <joint_name>${namespace}_cgo3_vertical_arm_joint</joint_name>
           </channel>
           <channel name="left_leg">
@@ -299,5 +299,5 @@
               <cmdMin>-6</cmdMin>
             </joint_control_pid>
-            <joint_name>${namespace}::${namespace}_left_leg_joint</joint_name>
+            <joint_name>${namespace}_left_leg_joint</joint_name>
           </channel>
           <channel name="right_leg">

File: models/typhoon_h480/urdf/multirotor_base.xacro (robot description, xacro)
@@ -38,78 +38,20 @@
     </gazebo>
     <gazebo reference="${robot_namespace}_left_leg">
-      <collision name="${robot_namespace}_collision">
-        <surface>
-          <friction>
-            <ode>
-              <mu>1</mu>
-              <mu2>1</mu2>
-            </ode>
-          </friction>
-          <contact>
-            <ode>
-              <kp>1e+8</kp>
-              <kd>1</kd>
-              <max_vel>0.01</max_vel>
-              <min_depth>0.001</min_depth>
-            </ode>
-          </contact>
-        </surface>
-      </collision>
-      <collision name="${robot_namespace}_collision_bar">
-        <surface>
-          <friction>
-            <ode>
-              <mu>1</mu>
-              <mu2>1</mu2>
-            </ode>
-          </friction>
-          <contact>
-            <ode>
-              <kp>1e+8</kp>
-              <kd>1</kd>
-              <max_vel>0.01</max_vel>
-              <min_depth>0.001</min_depth>
-            </ode>
-          </contact>
-        </surface>
-      </collision>
+      <mu1>1</mu1>
+      <mu2>1</mu2>
+      <kp>1e+8</kp>
+      <kd>1</kd>
+      <maxVel>0.01</maxVel>
+      <minDepth>0.001</minDepth>
+      <material>Gazebo/Grey</material>
     </gazebo>
     <gazebo reference="${robot_namespace}_right_leg">
-      <collision name="${robot_namespace}_collision">
-        <surface>
-          <friction>
-            <ode>
-              <mu>1</mu>
-              <mu2>1</mu2>
-            </ode>
-          </friction>
-          <contact>
-            <ode>
-              <kp>1e+8</kp>
-              <kd>1</kd>
-              <max_vel>0.01</max_vel>
-              <min_depth>0.001</min_depth>
-            </ode>
-          </contact>
-        </surface>
-      </collision>
-      <collision name="${robot_namespace}_collision_bar">
-        <surface>
-          <friction>
-            <ode>
-              <mu>1</mu>
-              <mu2>1</mu2>
-            </ode>
-          </friction>
-          <contact>
-            <ode>
-              <kp>1e+8</kp>
-              <kd>1</kd>
-              <max_vel>0.01</max_vel>
-              <min_depth>0.001</min_depth>
-            </ode>
-          </contact>
-        </surface>
-      </collision>
+      <mu1>1</mu1>
+      <mu2>1</mu2>
+      <kp>1e+8</kp>
+      <kd>1</kd>
+      <maxVel>0.01</maxVel>
+      <minDepth>0.001</minDepth>
+      <material>Gazebo/Grey</material>
     </gazebo>
     <link name="${robot_namespace}_left_leg">
@@ -119,5 +61,5 @@
         <inertia ixx="0.001" ixy="0" ixz="0" iyy="0.001" iyz="0" izz="0.001"/>
       </inertial>
-      <collision name="${robot_namespace}_collision">
+      <collision>
         <origin rpy="0 1.56893  0" xyz="-0.00526 -0.10262 -0.15925"/>
         <geometry>
@@ -125,5 +67,5 @@
         </geometry>
       </collision>
-      <collision name="${robot_namespace}_collision_bar">
+      <collision>
         <origin rpy="-0.501318 0 0" xyz="0.00025 -0.04451 -0.07318"/>
         <geometry>
@@ -131,5 +73,5 @@
         </geometry>
       </collision>
-      <visual name="${robot_namespace}_base_link_left_leg">
+      <visual>
         <origin rpy="0 0 0" xyz="-0.00025  0.04051  0.048"/>
         <geometry>
@@ -144,5 +86,5 @@
         <inertia ixx="0.001" ixy="0" ixz="0" iyy="0.001" iyz="0" izz="0.001"/>
       </inertial>
-      <collision name="${robot_namespace}_collision">
+      <collision>
         <origin rpy="0 1.56893 0" xyz="-0.00526  0.10262 -0.15925"/>
         <geometry>
@@ -150,5 +92,5 @@
         </geometry>
       </collision>
-      <collision name="${robot_namespace}_collision_bar">
+      <collision>
         <origin rpy="0.501318 0 0" xyz="0.00025  0.04451 -0.07318"/>
         <geometry>
@@ -156,5 +98,5 @@
         </geometry>
       </collision>
-      <visual name="${robot_namespace}_base_link_right_leg">
+      <visual>
         <origin rpy="0  0  0" xyz="-0.00025 -0.04051  0.048"/>
         <geometry>
@@ -181,11 +123,11 @@
     <gazebo reference="${robot_namespace}_left_leg_joint">
       <implicitSpringDamper>1</implicitSpringDamper>
-      <springStiffness>100000000</springStiffness>
-      <preserveFixedJoint>false</preserveFixedJoint>
+      <stopErp>0</stopErp>
+      <stopCfm>0</stopCfm>
     </gazebo>
     <gazebo reference="${robot_namespace}_right_leg_joint">
       <implicitSpringDamper>1</implicitSpringDamper>
-      <springStiffness>100000000</springStiffness>
-      <preserveFixedJoint>false</preserveFixedJoint>
+      <stopErp>0</stopErp>
+      <stopCfm>0</stopCfm>
     </gazebo>
     <link name="${robot_namespace}_cgo3_mount_link">
@@ -195,5 +137,5 @@
         <inertia ixx="0.001" ixy="0" ixz="0" iyy="0.001" iyz="0" izz="0.001"/>
       </inertial>
-      <visual name="typhoon_h480__cgo3_mount_visual">
+      <visual>
         <origin rpy="0 0 0" xyz="0 0 0"/>
         <geometry>
@@ -202,4 +144,7 @@
       </visual>
     </link>
+    <gazebo reference="${robot_namespace}_cgo3_mount_link">
+      <material>Gazebo/Grey</material>
+    </gazebo>
     <joint name="${robot_namespace}_cgo3_mount_joint" type="fixed">
       <parent link="${robot_namespace}_base_link"/>
@@ -219,5 +164,5 @@
         <inertia ixx="0.001" ixy="0" ixz="0" iyy="0.001" iyz="0" izz="0.001"/>
       </inertial>
-      <visual name="typhoon_h480__cgo3_vertical_arm_visual">
+      <visual>
         <origin rpy="0 0 0" xyz="0.026 0 0.1"/>
         <geometry>
@@ -226,4 +171,7 @@
       </visual>
     </link>
+    <gazebo reference="${robot_namespace}_cgo3_vertical_arm_link">
+      <material>Gazebo/Grey</material>
+    </gazebo>
     <joint name="${robot_namespace}_cgo3_vertical_arm_joint" type="revolute">
       <parent link="${robot_namespace}_cgo3_mount_link"/>
@@ -245,5 +193,5 @@
         <inertia ixx="0.001" ixy="0" ixz="0" iyy="0.001" iyz="0" izz="0.001"/>
       </inertial>
-      <visual name="typhoon_h480__cgo3_horizontal_arm_visual">
+      <visual>
         <origin rpy="0  0  0" xyz="-0.026  0     0.162"/>
         <geometry>
@@ -252,4 +200,7 @@
       </visual>
     </link>
+    <gazebo reference="${robot_namespace}_cgo3_horizontal_arm_link">
+      <material>Gazebo/Grey</material>
+    </gazebo>
     <joint name="${robot_namespace}_cgo3_horizontal_arm_joint" type="revolute">
       <parent link="${robot_namespace}_cgo3_vertical_arm_link"/>
@@ -271,5 +222,5 @@
         <inertia ixx="0.001" ixy="0" ixz="0" iyy="0.001" iyz="0" izz="0.001"/>
       </inertial>
-      <collision name="${robot_namespace}_cgo3_camera_collision">
+      <collision>
         <origin rpy="0  0  0" xyz="0   -0.03  0"/>
         <geometry>
@@ -277,5 +228,5 @@
         </geometry>
       </collision>
-      <visual name="${robot_namespace}_cgo3_camera_visual">
+      <visual>
         <origin rpy="0  0  0" xyz="0.041 -0.03   0.162"/>
         <geometry>
@@ -325,10 +276,17 @@
       <dynamics damping="0.1"/>
     </joint>
+    <gazebo reference="${robot_namespace}_cgo3_camera_link">
+      <mu1>1</mu1>
+      <mu2>1</mu2>
+      <kp>1e+8</kp>
+      <kd>1</kd>
+      <maxVel>0.01</maxVel>
+      <minDepth>0.001</minDepth>
+      <material>Gazebo/Black</material>
+    </gazebo>
     <gazebo reference="${robot_namespace}_cgo3_camera_joint">
       <implicitSpringDamper>1</implicitSpringDamper>
       <stopCfm>0.1</stopCfm>
       <stopErp>0.2</stopErp>
-      <mu1>1</mu1>
-      <mu2>1</mu2>
     </gazebo>
     <gazebo>
@@ -388,17 +346,6 @@
     <gazebo reference="${robot_namespace}_base_link">
       <material>Gazebo/${color}</material>
-      <collision name='base_link_inertia_collision'>
-        <surface>
-          <contact>
-            <ode>
-              <min_depth>0.001</min_depth>
-              <max_vel>0.0</max_vel>
-            </ode>
-          </contact>
-          <friction>
-            <ode/>
-          </friction>
-        </surface>
-      </collision>
+      <minDepth>0.001</minDepth>
+      <maxVel>0.0</maxVel>
    </gazebo>
   </xacro:macro>
