Commit message: rework typhoon URDF

File: models/typhoon_h480/urdf/multirotor_base.xacro (robot description, xacro)
@@ -12,9 +12,9 @@
       <inertial>
         <mass value="${mass}" />  <!-- [kg] -->
-        <origin rpy="0 0 0" xyz="0.001  0 -0.009"/>
+        <origin rpy="0 0 0" xyz="0.001005 0 -0.0090035"/>
         <xacro:insert_block name="inertia" />
       </inertial>
       <visual>
-        <origin rpy="0 0 -3.14159" xyz="0 0 0.26"/>
+        <origin rpy="0 0 3.14159" xyz="0 0 0.26"/>
         <geometry>
           <mesh filename="package://$(arg ros_package)typhoon_h480/meshes/${mesh_file}"
@@ -37,4 +37,156 @@
       <material>Gazebo/${color}</material>
     </gazebo>
+    <gazebo reference="${robot_namespace}_left_leg">
+      <collision name="${robot_namespace}_collision">
+        <surface>
+          <friction>
+            <ode>
+              <mu>1</mu>
+              <mu2>1</mu2>
+            </ode>
+          </friction>
+          <contact>
+            <ode>
+              <kp>1e+8</kp>
+              <kd>1</kd>
+              <max_vel>0.01</max_vel>
+              <min_depth>0.001</min_depth>
+            </ode>
+          </contact>
+        </surface>
+      </collision>
+      <collision name="${robot_namespace}_collision_bar">
+        <surface>
+          <friction>
+            <ode>
+              <mu>1</mu>
+              <mu2>1</mu2>
+            </ode>
+          </friction>
+          <contact>
+            <ode>
+              <kp>1e+8</kp>
+              <kd>1</kd>
+              <max_vel>0.01</max_vel>
+              <min_depth>0.001</min_depth>
+            </ode>
+          </contact>
+        </surface>
+      </collision>
+    </gazebo>
+    <gazebo reference="${robot_namespace}_right_leg">
+      <collision name="${robot_namespace}_collision">
+        <surface>
+          <friction>
+            <ode>
+              <mu>1</mu>
+              <mu2>1</mu2>
+            </ode>
+          </friction>
+          <contact>
+            <ode>
+              <kp>1e+8</kp>
+              <kd>1</kd>
+              <max_vel>0.01</max_vel>
+              <min_depth>0.001</min_depth>
+            </ode>
+          </contact>
+        </surface>
+      </collision>
+      <collision name="${robot_namespace}_collision_bar">
+        <surface>
+          <friction>
+            <ode>
+              <mu>1</mu>
+              <mu2>1</mu2>
+            </ode>
+          </friction>
+          <contact>
+            <ode>
+              <kp>1e+8</kp>
+              <kd>1</kd>
+              <max_vel>0.01</max_vel>
+              <min_depth>0.001</min_depth>
+            </ode>
+          </contact>
+        </surface>
+      </collision>
+    </gazebo>
+    <link name="${robot_namespace}_left_leg">
+      <inertial>
+        <mass value="0.1"/>
+        <origin rpy="0  0  0" xyz="0 -0.14313 -0.20725"/>
+        <inertia ixx="0.001" ixy="0" ixz="0" iyy="0.001" iyz="0" izz="0.001"/>
+      </inertial>
+      <collision name="${robot_namespace}_collision">
+        <origin rpy="0 1.56893  0" xyz="-0.00526 -0.10262 -0.15925"/>
+        <geometry>
+          <cylinder length="0.3" radius="0.012209"/>
+        </geometry>
+      </collision>
+      <collision name="${robot_namespace}_collision_bar">
+        <origin rpy="-0.501318 0 0" xyz="0.00025 -0.04451 -0.07318"/>
+        <geometry>
+          <cylinder length="0.176893" radius="0.00914984"/>
+        </geometry>
+      </collision>
+      <visual name="${robot_namespace}_base_link_left_leg">
+        <origin rpy="0 0 0" xyz="-0.00025  0.04051  0.048"/>
+        <geometry>
+          <mesh filename="package://$(arg ros_package)typhoon_h480/meshes/leg2_remeshed_v3.stl" scale="0.001 0.001 0.001"/>
+        </geometry>
+      </visual>
+    </link>
+    <link name="${robot_namespace}_right_leg">
+      <inertial>
+        <mass value="0.1"/>
+        <origin rpy="0 0 0" xyz="0 0.14314 -0.207252"/>
+        <inertia ixx="0.001" ixy="0" ixz="0" iyy="0.001" iyz="0" izz="0.001"/>
+      </inertial>
+      <collision name="${robot_namespace}_collision">
+        <origin rpy="0 1.56893 0" xyz="-0.00526  0.10262 -0.15925"/>
+        <geometry>
+          <cylinder length="0.3" radius="0.012209"/>
+        </geometry>
+      </collision>
+      <collision name="${robot_namespace}_collision_bar">
+        <origin rpy="0.501318 0 0" xyz="0.00025  0.04451 -0.07318"/>
+        <geometry>
+          <cylinder length="0.176893" radius="0.00914984"/>
+        </geometry>
+      </collision>
+      <visual name="${robot_namespace}_base_link_right_leg">
+        <origin rpy="0  0  0" xyz="-0.00025 -0.04051  0.048"/>
+        <geometry>
+          <mesh filename="package://$(arg ros_package)typhoon_h480/meshes/leg1_remeshed_v3.stl" scale="0.001 0.001 0.001"/>
+        </geometry>
+      </visual>
+    </link>
+    <joint name="${robot_namespace}_left_leg_joint" type="revolute">
+      <parent link="${robot_namespace}_base_link"/>
+      <child link="${robot_namespace}_left_leg"/>
+      <origin rpy="0 0 -3.14159" xyz="-0.00025  0.04051  0.212"/>
+      <axis xyz="-1 0 0"/>
+      <limit effort="100.0" lower="0.0" upper="1.0" velocity="-1.0"/>
+      <dynamics damping="1"/>
+    </joint>
+    <joint name="${robot_namespace}_right_leg_joint" type="revolute">
+      <parent link="${robot_namespace}_base_link"/>
+      <child link="${robot_namespace}_right_leg"/>
+      <origin rpy="0 0 -3.14159" xyz="-0.00025 -0.04051  0.212"/>
+      <axis xyz="1 0 0"/>
+      <limit effort="100.0" lower="0.0" upper="1.0" velocity="-1.0"/>
+      <dynamics damping="1"/>
+    </joint>
+    <gazebo reference="${robot_namespace}_left_leg_joint">
+      <implicitSpringDamper>1</implicitSpringDamper>
+      <springStiffness>100000000</springStiffness>
+      <preserveFixedJoint>false</preserveFixedJoint>
+    </gazebo>
+    <gazebo reference="${robot_namespace}_right_leg_joint">
+      <implicitSpringDamper>1</implicitSpringDamper>
+      <springStiffness>100000000</springStiffness>
+      <preserveFixedJoint>false</preserveFixedJoint>
+    </gazebo>
     <link name="${robot_namespace}_cgo3_mount_link">
       <inertial>
@@ -47,17 +199,4 @@
         <geometry>
           <mesh filename="package://$(arg ros_package)typhoon_h480/meshes/cgo3_mount_remeshed_v1.stl" scale="0.001 0.001 0.001"/>
-        </geometry>
-      </visual>
-    </link>
-    <link name="${robot_namespace}_cgo3_vertical_arm_link">
-      <inertial>
-        <mass value="0.1"/>
-        <origin rpy="0 0 0" xyz="-0.041 0 -0.162"/>
-        <inertia ixx="0.001" ixy="0" ixz="0" iyy="0.001" iyz="0" izz="0.001"/>
-      </inertial>
-      <visual name="typhoon_h480__cgo3_vertical_arm_visual">
-        <origin rpy="0 0 0" xyz="0.026 0 0.1"/>
-        <geometry>
-          <mesh filename="package://$(arg ros_package)typhoon_h480/meshes/cgo3_vertical_arm_remeshed_v1.stl" scale="0.001 0.001 0.001"/>
         </geometry>
       </visual>
@@ -66,8 +205,25 @@
       <parent link="${robot_namespace}_base_link"/>
       <child link="${robot_namespace}_cgo3_mount_link"/>
-      <origin rpy="0       0      -3.14159" xyz="0    0    0.26"/>
+      <origin rpy="0 0 -3.14159" xyz="0 0 0.26"/>
       <axis xyz="0  0  1"/>
       <limit effort="100.0" lower="0.0" upper="0.0" velocity="-1.0"/>
-    </joint>
+      <dynamics damping="1"/>
+    </joint>
+    <gazebo reference="${robot_namespace}_cgo3_mount_joint">
+      <implicitSpringDamper>1</implicitSpringDamper>
+    </gazebo>
+    <link name="${robot_namespace}_cgo3_vertical_arm_link">
+      <inertial>
+        <mass value="0.1"/>
+        <origin rpy="0 0 0" xyz="-0.041 0 -0.162"/>
+        <inertia ixx="0.001" ixy="0" ixz="0" iyy="0.001" iyz="0" izz="0.001"/>
+      </inertial>
+      <visual name="typhoon_h480__cgo3_vertical_arm_visual">
+        <origin rpy="0 0 0" xyz="0.026 0 0.1"/>
+        <geometry>
+          <mesh filename="package://$(arg ros_package)typhoon_h480/meshes/cgo3_vertical_arm_remeshed_v1.stl" scale="0.001 0.001 0.001"/>
+        </geometry>
+      </visual>
+    </link>
     <joint name="${robot_namespace}_cgo3_vertical_arm_joint" type="revolute">
       <parent link="${robot_namespace}_cgo3_mount_link"/>
@@ -76,55 +232,11 @@
       <axis xyz="0 0 1"/>
       <limit effort="100.0" lower="-1e+16" upper="1e+16" velocity="-1.0"/>
-    </joint>
-    <link name="${robot_namespace}_left_leg">
-      <inertial>
-        <mass value="0.1"/>
-        <origin rpy="0  0  0" xyz="0      -0.14313 -0.20725"/>
-        <inertia ixx="0.001" ixy="0" ixz="0" iyy="0.001" iyz="0" izz="0.001"/>
-      </inertial>
-      <collision name="typhoon_h480__collision">
-        <origin rpy="0       1.56893  0" xyz="-0.00526 -0.10262 -0.15925"/>
-        <geometry>
-          <cylinder length="0.3" radius="0.012209"/>
-        </geometry>
-      </collision>
-      <collision name="typhoon_h480__collision_bar">
-        <origin rpy="-0.50131  0       0" xyz="0.00025 -0.04451 -0.07318"/>
-        <geometry>
-          <cylinder length="0.176893" radius="0.00914984"/>
-        </geometry>
-      </collision>
-      <visual name="typhoon_h480__base_link_left_leg">
-        <origin rpy="0  0  0" xyz="-0.00025  0.04051  0.048"/>
-        <geometry>
-          <mesh filename="package://$(arg ros_package)typhoon_h480/meshes/leg2_remeshed_v3.stl" scale="0.001 0.001 0.001"/>
-        </geometry>
-      </visual>
-    </link>
-    <link name="${robot_namespace}_right_leg">
-      <inertial>
-        <mass value="0.1"/>
-        <origin rpy="0  0  0" xyz="0       0.14313 -0.20725"/>
-        <inertia ixx="0.001" ixy="0" ixz="0" iyy="0.001" iyz="0" izz="0.001"/>
-      </inertial>
-      <collision name="typhoon_h480__collision">
-        <origin rpy="0       1.56893  0" xyz="-0.00526  0.10262 -0.15925"/>
-        <geometry>
-          <cylinder length="0.3" radius="0.012209"/>
-        </geometry>
-      </collision>
-      <collision name="typhoon_h480__collision_bar">
-        <origin rpy="0.50131  0       0" xyz="0.00025  0.04451 -0.07318"/>
-        <geometry>
-          <cylinder length="0.176893" radius="0.00914984"/>
-        </geometry>
-      </collision>
-      <visual name="typhoon_h480__base_link_right_leg">
-        <origin rpy="0  0  0" xyz="-0.00025 -0.04051  0.048"/>
-        <geometry>
-          <mesh filename="package://$(arg ros_package)typhoon_h480/meshes/leg1_remeshed_v3.stl" scale="0.001 0.001 0.001"/>
-        </geometry>
-      </visual>
-    </link>
+      <dynamics damping="0.1"/>
+    </joint>
+    <gazebo reference="${robot_namespace}_cgo3_vertical_arm_joint">
+      <implicitSpringDamper>1</implicitSpringDamper>
+      <stopCfm>0.1</stopCfm>
+      <stopErp>0.2</stopErp>
+    </gazebo>
     <link name="${robot_namespace}_cgo3_horizontal_arm_link">
       <inertial>
@@ -140,4 +252,17 @@
       </visual>
     </link>
+    <joint name="${robot_namespace}_cgo3_horizontal_arm_joint" type="revolute">
+      <parent link="${robot_namespace}_cgo3_vertical_arm_link"/>
+      <child link="${robot_namespace}_cgo3_horizontal_arm_link"/>
+      <origin rpy="0  0  0" xyz="0.052  0    -0.062"/>
+      <axis xyz="-1  0  0"/>
+      <limit effort="100.0" lower="-0.785398" upper="0.785398" velocity="-1.0"/>
+      <dynamics damping="0.1"/>
+    </joint>
+    <gazebo reference="${robot_namespace}_cgo3_horizontal_arm_joint">
+      <implicitSpringDamper>1</implicitSpringDamper>
+      <stopCfm>0.1</stopCfm>
+      <stopErp>0.2</stopErp>
+    </gazebo>
     <link name="${robot_namespace}_cgo3_camera_link">
       <inertial>
@@ -146,5 +271,5 @@
         <inertia ixx="0.001" ixy="0" ixz="0" iyy="0.001" iyz="0" izz="0.001"/>
       </inertial>
-      <collision name="typhoon_h480__cgo3_camera_collision">
+      <collision name="${robot_namespace}_cgo3_camera_collision">
         <origin rpy="0  0  0" xyz="0   -0.03  0"/>
         <geometry>
@@ -152,5 +277,5 @@
         </geometry>
       </collision>
-      <visual name="typhoon_h480__cgo3_camera_visual">
+      <visual name="${robot_namespace}_cgo3_camera_visual">
         <origin rpy="0  0  0" xyz="0.041 -0.03   0.162"/>
         <geometry>
@@ -160,22 +285,4 @@
     </link>
     <gazebo reference="${robot_namespace}_cgo3_camera_link">
-      <collision name='typhoon_h480__cgo3_camera_collision'>
-        <surface>
-          <friction>
-            <ode>
-              <mu>1</mu>
-              <mu2>1</mu2>
-            </ode>
-          </friction>
-          <contact>
-            <ode>
-              <kp>1e+8</kp>
-              <kd>1</kd>
-              <max_vel>0.01</max_vel>
-              <min_depth>0.001</min_depth>
-            </ode>
-          </contact>
-        </surface>
-      </collision>
       <sensor name="camera_imu" type="imu">
         <always_on>1</always_on>
@@ -210,11 +317,4 @@
       </sensor>
     </gazebo>
-    <joint name="${robot_namespace}_cgo3_horizontal_arm_joint" type="revolute">
-      <parent link="${robot_namespace}_cgo3_vertical_arm_link"/>
-      <child link="${robot_namespace}_cgo3_horizontal_arm_link"/>
-      <origin rpy="0  0  0" xyz="0.052  0    -0.062"/>
-      <axis xyz="-1  0  0"/>
-      <limit effort="100.0" lower="-0.785398" upper="0.785398" velocity="-1.0"/>
-    </joint>
     <joint name="${robot_namespace}_cgo3_camera_joint" type="revolute">
       <parent link="${robot_namespace}_cgo3_horizontal_arm_link"/>
@@ -223,25 +323,18 @@
       <axis xyz="0 -1  0"/>
       <limit effort="100.0" lower="-1.05" upper="2.09" velocity="-1.0"/>
-    </joint>
-    <joint name="${robot_namespace}_left_leg_joint" type="revolute">
-      <parent link="${robot_namespace}_base_link"/>
-      <child link="${robot_namespace}_left_leg"/>
-      <origin rpy="0 0 -3.14159" xyz="-0.00025 0.04051 0.212"/>
-      <axis xyz="-1 0 0"/>
-      <limit effort="100.0" lower="0.0" upper="1.0" velocity="-1.0"/>
-    </joint>
-    <joint name="${robot_namespace}_right_leg_joint" type="revolute">
-      <parent link="${robot_namespace}_base_link"/>
-      <child link="${robot_namespace}_right_leg"/>
-      <origin rpy="0 0 -3.14159" xyz="-0.00025 -0.04051 0.212"/>
-      <axis xyz="1 0 0"/>
-      <limit effort="100.0" lower="0.0" upper="1.0" velocity="-1.0"/>
-    </joint>
-    <!-- attach multirotor_base_plugin to the base_link -->
+      <dynamics damping="0.1"/>
+    </joint>
+    <gazebo reference="${robot_namespace}_cgo3_camera_joint">
+      <implicitSpringDamper>1</implicitSpringDamper>
+      <stopCfm>0.1</stopCfm>
+      <stopErp>0.2</stopErp>
+      <mu1>1</mu1>
+      <mu2>1</mu2>
+    </gazebo>
     <gazebo>
       <plugin name='gimbal_controller' filename='libgazebo_gimbal_controller_plugin.so'>
         <joint_yaw>${namespace}::${namespace}_cgo3_vertical_arm_joint</joint_yaw>
-        <joint_roll>${namespace}::${namespace}_cgo3_horizontal_arm_joint</joint_roll>
-        <joint_pitch>${namespace}::${namespace}_cgo3_camera_joint</joint_pitch>
+        <joint_roll>${namespace}::${namespace}_cgo3_camera_joint</joint_roll>
+        <joint_pitch>${namespace}::${namespace}_cgo3_horizontal_arm_joint</joint_pitch>
         <control_gimbal_channels>
           <channel>
@@ -284,4 +377,7 @@
         <gimbal_imu>camera_imu</gimbal_imu>
       </plugin>
+    </gazebo>
+    <!-- attach multirotor_base_plugin to the base_link -->
+    <gazebo>
       <plugin filename="libgazebo_multirotor_base_plugin.so" name="rosbag">
         <robotNamespace>${robot_namespace}</robotNamespace>

File: models/typhoon_h480/urdf/typhoon_h480.xacro (robot description, xacro)
@@ -72,6 +72,6 @@
     mesh_scale="${mesh_scale_prop}"
     color="DarkGrey">
-    <origin xyz="0.20939 -0.12276  0.34221" rpy="0 0 -1.04719" />
-    <axis xyz="0.02558 -0.04272  0.99875"/>
+    <origin xyz="0.00187 -0.2427   0.34221" rpy="0 0 -3.14159" />
+    <axis xyz="-5.03300000e-02  -1.50000000e-04   9.98730000e-01"/>
     <xacro:insert_block name="rotor_inertia" />
   </xacro:vertical_rotor>
@@ -94,6 +94,6 @@
     mesh_scale="${mesh_scale_prop}"
     color="Blue">
-    <origin xyz="-0.21139  0.11976  0.34221" rpy="0 0 1.04719" />
-    <axis xyz="-4.97500000e-02   8.10000000e-04   9.98760000e-01"/>
+    <origin xyz="0.00187  0.2427   0.34221" rpy="0 0 1.04719" />
+    <axis xyz="-0.033996 -0.0006 0.68216"/>
     <xacro:insert_block name="rotor_inertia" />
   </xacro:vertical_rotor>
@@ -116,5 +116,5 @@
     color="DarkGrey">
     <origin xyz="0.20939  0.12276  0.34221" rpy="0 0 -1.04719" />
-    <axis xyz="-0.05055  0.00463  0.99871"/>
+    <axis xyz="0.0404 -0.0876 1.8976"/>
     <xacro:insert_block name="rotor_inertia" />
   </xacro:vertical_rotor>
@@ -137,5 +137,5 @@
     color="Blue">
     <origin xyz="-0.21139 -0.11976  0.34221" rpy="0 0 -3.14159" />
-    <axis xyz="0.02347 -0.04342  0.99878"/>
+    <axis xyz="0.0446 -0.0825 1.8977"/>
     <xacro:insert_block name="rotor_inertia" />
   </xacro:vertical_rotor>
@@ -157,6 +157,6 @@
     mesh_scale="${mesh_scale_prop}"
     color="Blue">
-    <origin rpy="0 0 -3.14159" xyz="0.00187 -0.2427 0.34221"/>
-    <axis xyz="-5.03300000e-02 -1.50000000e-04 9.98730000e-01"/>
+    <origin rpy="0 0 -1.04719" xyz="0.20939 -0.12276  0.34221"/>
+    <axis xyz="0.02558 -0.04272  0.99875"/>
     <xacro:insert_block name="rotor_inertia" />
   </xacro:vertical_rotor>
@@ -178,6 +178,6 @@
     mesh_scale="${mesh_scale_prop}"
     color="DarkGrey">
-    <origin rpy="0 0 1.04719" xyz="0.00187 0.2427 0.34221"/>
-    <axis xyz="0.02564 -0.04266 0.99876"/>
+    <origin rpy="0 0 1.04719" xyz="-0.21139  0.11976  0.34221"/>
+    <axis xyz="0.0486 0.0811 1.8976"/>
     <xacro:insert_block name="rotor_inertia" />
   </xacro:vertical_rotor>

Commit message: typhoon adding camera_udp_port and colors

File: models/typhoon_h480/urdf/multirotor_base.xacro (robot description, xacro)
@@ -2,5 +2,5 @@
   <!-- Main multirotor link -->
   <xacro:macro name="multirotor_base_macro"
-    params="robot_namespace mass body_width body_height mesh_file mesh_scale color *inertia">
+    params="robot_namespace mass body_width body_height camera_udp_port mesh_file mesh_scale color *inertia">
     <link name="${robot_namespace}_base_link"></link>
     <joint name="${robot_namespace}_base_joint" type="fixed">
@@ -78,4 +78,7 @@
           <mesh filename="package://$(arg ros_package)typhoon_h480/meshes/leg2_remeshed_v3.stl" scale="0.001 0.001 0.001"/>
         </geometry>
+        <material name="Gazebo/Grey">
+          <color rgba="0.5 0.5 0.5 1"/>
+        </material>
       </visual>
     </link>
@@ -103,4 +106,7 @@
           <mesh filename="package://$(arg ros_package)typhoon_h480/meshes/leg1_remeshed_v3.stl" scale="0.001 0.001 0.001"/>
         </geometry>
+        <material name="Gazebo/Grey">
+          <color rgba="0.5 0.5 0.5 1"/>
+        </material>
       </visual>
     </link>
@@ -142,4 +148,7 @@
           <mesh filename="package://$(arg ros_package)typhoon_h480/meshes/cgo3_mount_remeshed_v1.stl" scale="0.001 0.001 0.001"/>
         </geometry>
+        <material name="Gazebo/Grey">
+          <color rgba="0.5 0.5 0.5 1"/>
+        </material>
       </visual>
     </link>
@@ -169,4 +178,7 @@
           <mesh filename="package://$(arg ros_package)typhoon_h480/meshes/cgo3_vertical_arm_remeshed_v1.stl" scale="0.001 0.001 0.001"/>
         </geometry>
+        <material name="Gazebo/Grey">
+          <color rgba="0.5 0.5 0.5 1"/>
+        </material>
       </visual>
     </link>
@@ -198,4 +210,7 @@
           <mesh filename="package://$(arg ros_package)typhoon_h480/meshes/cgo3_horizontal_arm_remeshed_v1.stl" scale="0.001 0.001 0.001"/>
         </geometry>
+        <material name="Gazebo/Grey">
+          <color rgba="0.5 0.5 0.5 1"/>
+        </material>
       </visual>
     </link>
@@ -233,4 +248,7 @@
           <mesh filename="package://$(arg ros_package)typhoon_h480/meshes/cgo3_camera_remeshed_v1.stl" scale="0.001 0.001 0.001"/>
         </geometry>
+        <material name="Gazebo/Black">
+          <color rgba="0. 0. 0. 1"/>
+        </material>
       </visual>
     </link>
@@ -241,5 +259,5 @@
       <sensor name="camera" type="camera">
         <pose>0 -0.03 0 0 0 3.14159</pose>
-        <camera>
+        <camera name='__default__'>>
           <horizontal_fov>2.0</horizontal_fov>
           <image>
@@ -254,9 +272,9 @@
         </camera>
         <always_on>1</always_on>
-        <update_rate>10</update_rate>
+        <update_rate>30</update_rate>
         <visualize>true</visualize>
         <plugin name="GstCameraPlugin" filename="libgazebo_gst_camera_plugin.so">
             <robotNamespace></robotNamespace>
-            <udpPort>5600</udpPort>
+            <udpPort>$(arg camera_udp_port)</udpPort>
         </plugin>
       </sensor>
@@ -371,7 +389,13 @@
         <xacro:if value="${direction == 'ccw'}">
           <origin rpy="0  0  0" xyz="-0.21139 -0.11976 -0.08221"/>
+          <material name="Gazebo/Blue">
+            <color rgba="0. 0. 1. 1"/>
+          </material>
         </xacro:if>
         <xacro:if value="${direction == 'cw'}">
           <origin rpy="0  0  0" xyz="0.00187 -0.2427  -0.08221"/>
+          <material name="Gazebo/Grey">
+            <color rgba="0. 0. 0. 1"/>
+          </material>
         </xacro:if>
       </visual>

File: models/typhoon_h480/urdf/typhoon_h480.xacro (robot description, xacro)
@@ -50,4 +50,5 @@
     mesh_scale="${mesh_scale}"
     color="${color}"
+    camera_udp_port="$(arg camera_udp_port)"
     >
     <xacro:insert_block name="body_inertia" />

File: models/typhoon_h480/urdf/typhoon_h480_base.xacro (robot description, xacro)
@@ -31,4 +31,5 @@
   <xacro:arg name='enable_camera' default='false' />
   <xacro:arg name='log_file' default='iris' />
+  <xacro:arg name='camera_udp_port' default='5600' />
   <!-- macros for gazebo plugins, sensors -->
   <xacro:include filename="$(arg typhoon_dir)/urdf/component_snippets.xacro" />
