Commit message: Iris fixing package path for ros

File: models/rotors_description/urdf/iris_base.xacro (robot description, xacro)
@@ -5,4 +5,5 @@
   -->
   <xacro:arg name='name' default='iris' />
+  <xacro:arg name='ros_package' default='mavlink_sitl_gazebo/models/' />
   <xacro:arg name='mavlink_addr' default='INADDR_ANY' />
   <xacro:arg name='mavlink_udp_port' default='14560' />

File: models/rotors_description/urdf/multirotor_base.xacro (robot description, xacro)
@@ -35,5 +35,5 @@
         <origin xyz="0 0 0" rpy="0 0 0" />
         <geometry>
-          <mesh filename="package://rotors_description/meshes/${mesh_file}"
+          <mesh filename="package://$(arg ros_package)rotors_description/meshes/${mesh_file}"
             scale="${mesh_scale}" />
           <!-- <box size="${body_width} ${body_width} ${body_height}"/> --> <!-- [m] [m] [m] -->
@@ -95,5 +95,5 @@
           <!-- <cylinder length="0.005" radius="${radius_rotor}"/> --> <!-- [m] -->
           <!-- <mesh filename="package://rotors_description/meshes/propeller_${direction}.dae" -->
-          <mesh filename="package://rotors_description/meshes/${mesh}_${direction}.dae"
+          <mesh filename="package://$(arg ros_package)rotors_description/meshes/${mesh}_${direction}.dae"
             scale="${mesh_scale}" />
           <!-- <box size="${2*radius_rotor} 0.01 0.005"/> -->

Commit message: Removed ros_package from urdfs

File: models/rotors_description/urdf/iris_base.xacro (robot description, xacro)
@@ -5,5 +5,4 @@
   -->
   <xacro:arg name='name' default='iris' />
-  <xacro:arg name='ros_package' default='mavlink_sitl_gazebo/models/' />
   <xacro:arg name='mavlink_addr' default='INADDR_ANY' />
   <xacro:arg name='mavlink_udp_port' default='14560' />

File: models/rotors_description/urdf/multirotor_base.xacro (robot description, xacro)
@@ -35,5 +35,5 @@
         <origin xyz="0 0 0" rpy="0 0 0" />
         <geometry>
-          <mesh filename="package://$(arg ros_package)rotors_description/meshes/${mesh_file}"
+          <mesh filename="package://rotors_description/meshes/${mesh_file}"
             scale="${mesh_scale}" />
           <!-- <box size="${body_width} ${body_width} ${body_height}"/> --> <!-- [m] [m] [m] -->
@@ -101,5 +101,5 @@
           <!-- <cylinder length="0.005" radius="${radius_rotor}"/> --> <!-- [m] -->
           <!-- <mesh filename="package://rotors_description/meshes/propeller_${direction}.dae" -->
-          <mesh filename="package://$(arg ros_package)rotors_description/meshes/${mesh}_${direction}.dae"
+          <mesh filename="package://rotors_description/meshes/${mesh}_${direction}.dae"
             scale="${mesh_scale}" />
           <!-- <box size="${2*radius_rotor} 0.01 0.005"/> -->

File: models/typhoon_h480/urdf/multirotor_base.xacro (robot description, xacro)
@@ -18,5 +18,5 @@
         <origin rpy="0 0 3.14159" xyz="0 0 0.26"/>
         <geometry>
-          <mesh filename="package://$(arg ros_package)typhoon_h480/meshes/${mesh_file}"
+          <mesh filename="package://typhoon_h480/meshes/${mesh_file}"
             scale="${mesh_scale}" />
           <!-- <box size="${body_width} ${body_width} ${body_height}"/> --> <!-- [m] [m] [m] -->
@@ -76,5 +76,5 @@
         <origin rpy="0 0 0" xyz="-0.00025  0.04051  0.048"/>
         <geometry>
-          <mesh filename="package://$(arg ros_package)typhoon_h480/meshes/leg2_remeshed_v3.stl" scale="0.001 0.001 0.001"/>
+          <mesh filename="package://typhoon_h480/meshes/leg2_remeshed_v3.stl" scale="0.001 0.001 0.001"/>
         </geometry>
         <material name="Gazebo/Grey">
@@ -104,5 +104,5 @@
         <origin rpy="0  0  0" xyz="-0.00025 -0.04051  0.048"/>
         <geometry>
-          <mesh filename="package://$(arg ros_package)typhoon_h480/meshes/leg1_remeshed_v3.stl" scale="0.001 0.001 0.001"/>
+          <mesh filename="package://typhoon_h480/meshes/leg1_remeshed_v3.stl" scale="0.001 0.001 0.001"/>
         </geometry>
         <material name="Gazebo/Grey">
@@ -146,5 +146,5 @@
         <origin rpy="0 0 0" xyz="0 0 0"/>
         <geometry>
-          <mesh filename="package://$(arg ros_package)typhoon_h480/meshes/cgo3_mount_remeshed_v1.stl" scale="0.001 0.001 0.001"/>
+          <mesh filename="package://typhoon_h480/meshes/cgo3_mount_remeshed_v1.stl" scale="0.001 0.001 0.001"/>
         </geometry>
         <material name="Gazebo/Grey">
@@ -176,5 +176,5 @@
         <origin rpy="0 0 0" xyz="0.026 0 0.1"/>
         <geometry>
-          <mesh filename="package://$(arg ros_package)typhoon_h480/meshes/cgo3_vertical_arm_remeshed_v1.stl" scale="0.001 0.001 0.001"/>
+          <mesh filename="package://typhoon_h480/meshes/cgo3_vertical_arm_remeshed_v1.stl" scale="0.001 0.001 0.001"/>
         </geometry>
         <material name="Gazebo/Grey">
@@ -208,5 +208,5 @@
         <origin rpy="0  0  0" xyz="-0.026  0     0.162"/>
         <geometry>
-          <mesh filename="package://$(arg ros_package)typhoon_h480/meshes/cgo3_horizontal_arm_remeshed_v1.stl" scale="0.001 0.001 0.001"/>
+          <mesh filename="package://typhoon_h480/meshes/cgo3_horizontal_arm_remeshed_v1.stl" scale="0.001 0.001 0.001"/>
         </geometry>
         <material name="Gazebo/Grey">
@@ -246,5 +246,5 @@
         <origin rpy="0  0  0" xyz="0.041 -0.03   0.162"/>
         <geometry>
-          <mesh filename="package://$(arg ros_package)typhoon_h480/meshes/cgo3_camera_remeshed_v1.stl" scale="0.001 0.001 0.001"/>
+          <mesh filename="package://typhoon_h480/meshes/cgo3_camera_remeshed_v1.stl" scale="0.001 0.001 0.001"/>
         </geometry>
         <material name="Gazebo/Black">
@@ -384,5 +384,5 @@
       <visual>
         <geometry>
-          <mesh filename="package://$(arg ros_package)typhoon_h480/meshes/prop_${direction}_assembly_remeshed_v3.stl"
+          <mesh filename="package://typhoon_h480/meshes/prop_${direction}_assembly_remeshed_v3.stl"
             scale="${mesh_scale}" />
         </geometry>

File: models/typhoon_h480/urdf/typhoon_h480_base.xacro (robot description, xacro)
@@ -5,5 +5,4 @@
   -->
   <xacro:arg name='name' default='iris' />
-  <xacro:arg name='ros_package' default='mavlink_sitl_gazebo/models/' />
   <xacro:arg name='mavlink_addr' default='INADDR_ANY' />
   <xacro:arg name='mavlink_udp_port' default='14560' />
