Commit message: Use Gazebo GPS Sensor
Signed-off-by: Nicolae Rosia <nicolae.rosia@gmail.com>

File: models/rotors_description/urdf/component_snippets.xacro (robot description, xacro)
@@ -119,5 +119,5 @@
   </xacro:macro>
   <!-- Macro to add the mavlink interface. -->
-  <xacro:macro name="mavlink_interface_macro" params="namespace imu_sub_topic">
+  <xacro:macro name="mavlink_interface_macro" params="namespace imu_sub_topic gps_sub_topic">
     <gazebo>
       <plugin name="mavlink_interface" filename="librotors_gazebo_mavlink_interface.so">
@@ -125,4 +125,5 @@
         <imuSubTopic>${imu_sub_topic}</imuSubTopic>
         <motorSpeedCommandPubTopic>gazebo/command/motor_speed</motorSpeedCommandPubTopic>
+        <gpsPubTopic>${gps_sub_topic}</gpsPubTopic>
       </plugin>
     </gazebo>

File: models/rotors_description/urdf/iris_base.xacro (robot description, xacro)
@@ -2,4 +2,5 @@
 <robot name="iris" xmlns:xacro="http://ros.org/wiki/xacro">
   <xacro:include filename="$(arg rotors_description_dir)/urdf/component_snippets.xacro" />
+  <xacro:include filename="$(arg rotors_description_dir)/urdf/gazebo_gps.xacro" />
   <!-- Instantiate iris "mechanics" -->
   <xacro:include filename="$(arg rotors_description_dir)/urdf/iris.xacro" />
@@ -9,7 +10,16 @@
     namespace="${namespace}"
     imu_sub_topic="imu"
+    gps_sub_topic="/gazebo/default/iris/gps_link/gps"
     >
   </xacro:mavlink_interface_macro>
   </xacro:if>
+  <xacro:gazebo_gps
+    name="gps"
+    parent="base_link"
+    mass="0.015"
+  >
+    <inertia ixx="0.00001" ixy="0.0" ixz="0.0" iyy="0.00001" iyz="0.0" izz="0.00001" />
+    <origin xyz="0 0 0" rpy="0 0 0" />
+  </xacro:gazebo_gps>
   <!-- Mount an ADIS16448 IMU. -->
   <xacro:imu_plugin_macro

Commit message: Remove slowdown parameter
Signed-off-by: Nicolae Rosia <nicolae.rosia@gmail.com>

File: models/rotors_description/urdf/component_snippets.xacro (robot description, xacro)
@@ -19,5 +19,5 @@
   <!-- Macro to add logging to a bag file. -->
   <xacro:macro name="bag_plugin_macro"
-    params="namespace bag_file rotor_velocity_slowdown_sim">
+    params="namespace bag_file">
     <gazebo>
       <plugin filename="librotors_gazebo_bag_plugin.so" name="rosbag">
@@ -28,5 +28,4 @@
         <commandAttitudeThrustSubTopic>command/attitude</commandAttitudeThrustSubTopic>
         <commandAttitudeThrustPubTopic>command/attitude</commandAttitudeThrustPubTopic>
-        <rotorVelocitySlowdownSim>${rotor_velocity_slowdown_sim}</rotorVelocitySlowdownSim>
       </plugin>
     </gazebo>

File: models/rotors_description/urdf/iris.xacro (robot description, xacro)
@@ -3,5 +3,4 @@
   <!-- Properties -->
   <xacro:property name="namespace" value="iris" />
-  <xacro:property name="rotor_velocity_slowdown_sim" value="10" />
   <xacro:property name="mesh_file" value="iris.dae" />
   <xacro:property name="mesh_scale" value="1 1 1"/>
@@ -35,7 +34,7 @@
   <xacro:property name="rotor_inertia">
     <inertia
-    ixx="${1/12 * mass_rotor * (0.015 * 0.015 + 0.003 * 0.003) * rotor_velocity_slowdown_sim}"
-    iyy="${1/12 * mass_rotor * (4 * radius_rotor * radius_rotor + 0.003 * 0.003) * rotor_velocity_slowdown_sim}"
-    izz="${1/12 * mass_rotor * (4 * radius_rotor * radius_rotor + 0.015 * 0.015) * rotor_velocity_slowdown_sim}"
+    ixx="${1/12 * mass_rotor * (0.015 * 0.015 + 0.003 * 0.003)}"
+    iyy="${1/12 * mass_rotor * (4 * radius_rotor * radius_rotor + 0.003 * 0.003)}"
+    izz="${1/12 * mass_rotor * (4 * radius_rotor * radius_rotor + 0.015 * 0.015)}"
     ixy="0.0" ixz="0.0"  iyz="0.0" /> <!-- [kg.m^2] [kg.m^2] [kg.m^2] [kg.m^2] [kg.m^2] [kg.m^2] -->
   </xacro:property>

File: models/rotors_description/urdf/iris_base.xacro (robot description, xacro)
@@ -87,5 +87,4 @@
       namespace="${namespace}"
       bag_file="$(arg log_file)"
-      rotor_velocity_slowdown_sim="${rotor_velocity_slowdown_sim}"
     >
     </xacro:bag_plugin_macro>

File: models/rotors_description/urdf/multirotor_base.xacro (robot description, xacro)
@@ -52,5 +52,4 @@
         <robotNamespace>${robot_namespace}</robotNamespace>
         <linkName>base_link</linkName>
-        <rotorVelocitySlowdownSim>${rotor_velocity_slowdown_sim}</rotorVelocitySlowdownSim>
       </plugin>
     </gazebo>
@@ -109,5 +108,4 @@
         <rollingMomentCoefficient>${rolling_moment_coefficient}</rollingMomentCoefficient>
         <motorSpeedPubTopic>motor_speed/${motor_number}</motorSpeedPubTopic>
-        <rotorVelocitySlowdownSim>${rotor_velocity_slowdown_sim}</rotorVelocitySlowdownSim>
       </plugin>
     </gazebo>

Commit message: add mavlink_addr(INADDR_ANY) and mavlink_udp_port(14560) to rotors_description xacro for iris_base and in component_snippets xacros.

File: models/rotors_description/urdf/component_snippets.xacro (robot description, xacro)
@@ -119,9 +119,11 @@
   </xacro:macro>
   <!-- Macro to add the mavlink interface. -->
-  <xacro:macro name="mavlink_interface_macro" params="namespace imu_sub_topic">
+  <xacro:macro name="mavlink_interface_macro" params="namespace imu_sub_topic mavlink_addr mavlink_udp_port">
     <gazebo>
       <plugin name="mavlink_interface" filename="librotors_gazebo_mavlink_interface.so">
         <robotNamespace>${namespace}</robotNamespace>
         <imuSubTopic>${imu_sub_topic}</imuSubTopic>
+        <mavlink_addr>$(arg mavlink_addr)</mavlink_addr>
+        <mavlink_udp_port>$(arg mavlink_udp_port)</mavlink_udp_port>
         <motorSpeedCommandPubTopic>/gazebo/command/motor_speed</motorSpeedCommandPubTopic>
       </plugin>

File: models/rotors_description/urdf/iris_base.xacro (robot description, xacro)
@@ -9,4 +9,6 @@
     namespace="${namespace}"
     imu_sub_topic="/imu"
+    mavlink_addr="INADDR_ANY"
+    mavlink_udp_port="14560"
     >
   </xacro:mavlink_interface_macro>

Commit message: WIP

File: models/rotors_description/urdf/component_snippets.xacro (robot description, xacro)
@@ -128,5 +128,5 @@
   </xacro:macro>
   <!-- Macro to add the mavlink interface. -->
-  <xacro:macro name="mavlink_interface_macro" params="namespace imu_sub_topic gps_sub_topic mavlink_addr mavlink_udp_port serial_enabled serial_device baudrate qgc_addr qgc_udp_port hil_mode hil_state_level vehicle_is_tailsitter send_vision_estimation send_odometry">
+  <xacro:macro name="mavlink_interface_macro" params="namespace imu_sub_topic gps_sub_topic mavlink_addr mavlink_udp_port serial_enabled serial_device baudrate qgc_addr qgc_udp_port hil_mode hil_state_level vehicle_is_tailsitter send_vision_estimation send_odometry enable_lockstep">
     <gazebo>
       <plugin name="mavlink_interface" filename="libgazebo_mavlink_interface.so">
@@ -146,4 +146,5 @@
         <send_vision_estimation>$(arg send_vision_estimation)</send_vision_estimation>
         <send_odometry>$(arg send_odometry)</send_odometry>
+        <enable_lockstep>$(arg enable_lockstep)</enable_lockstep>
         <motorSpeedCommandPubTopic>/gazebo/command/motor_speed</motorSpeedCommandPubTopic>
         <control_channels>

File: models/rotors_description/urdf/iris_base.xacro (robot description, xacro)
@@ -16,4 +16,5 @@
   <xacro:arg name='send_vision_estimation' default='false' />
   <xacro:arg name='send_odometry' default='false' />
+  <xacro:arg name='enable_lockstep' default='true' />
   <xacro:arg name='vehicle_is_tailsitter' default='false' />
   <xacro:arg name='visual_material' default='DarkGrey' />
@@ -64,4 +65,5 @@
     send_vision_estimation="$(arg send_vision_estimation)"
     send_odometry="$(arg send_odometry)"
+    enable_lockstep="$(arg enable_lockstep)"
     >
   </xacro:mavlink_interface_macro>

Commit message: models: enable lockstep and TCP everywhere
Let's try this :).

File: models/rotors_description/urdf/component_snippets.xacro (robot description, xacro)
@@ -128,5 +128,5 @@
   </xacro:macro>
   <!-- Macro to add the mavlink interface. -->
-  <xacro:macro name="mavlink_interface_macro" params="namespace imu_sub_topic gps_sub_topic mavlink_addr mavlink_udp_port serial_enabled serial_device baudrate qgc_addr qgc_udp_port hil_mode hil_state_level vehicle_is_tailsitter send_vision_estimation send_odometry">
+  <xacro:macro name="mavlink_interface_macro" params="namespace imu_sub_topic gps_sub_topic mavlink_addr mavlink_udp_port serial_enabled serial_device baudrate qgc_addr qgc_udp_port hil_mode hil_state_level vehicle_is_tailsitter send_vision_estimation send_odometry enable_lockstep use_tcp">
     <gazebo>
       <plugin name="mavlink_interface" filename="libgazebo_mavlink_interface.so">
@@ -146,4 +146,6 @@
         <send_vision_estimation>$(arg send_vision_estimation)</send_vision_estimation>
         <send_odometry>$(arg send_odometry)</send_odometry>
+        <enable_lockstep>$(arg enable_lockstep)</enable_lockstep>
+        <use_tcp>$(arg use_tcp)</use_tcp>
         <motorSpeedCommandPubTopic>/gazebo/command/motor_speed</motorSpeedCommandPubTopic>
         <control_channels>

File: models/rotors_description/urdf/iris_base.xacro (robot description, xacro)
@@ -16,4 +16,6 @@
   <xacro:arg name='send_vision_estimation' default='false' />
   <xacro:arg name='send_odometry' default='false' />
+  <xacro:arg name='enable_lockstep' default='true' />
+  <xacro:arg name='use_tcp' default='true' />
   <xacro:arg name='vehicle_is_tailsitter' default='false' />
   <xacro:arg name='visual_material' default='DarkGrey' />
@@ -64,4 +66,6 @@
     send_vision_estimation="$(arg send_vision_estimation)"
     send_odometry="$(arg send_odometry)"
+    enable_lockstep="$(arg enable_lockstep)"
+    use_tcp="$(arg use_tcp)"
     >
   </xacro:mavlink_interface_macro>

Commit message: Adding the quadcopter plugin in urdf format

File: models/rotors_description/urdf/component_snippets.xacro (robot description, xacro)
@@ -115,4 +115,11 @@
         <imuSubTopic>/${imu_sub_topic}</imuSubTopic>
         <motorSpeedCommandPubTopic>/gazebo/command/motor_speed</motorSpeedCommandPubTopic>
+      </plugin>
+    </gazebo>
+  </xacro:macro>
+  <!-- Macro to add the reset the quadcopters. -->
+  <xacro:macro name="reset_plugin_macro" params="namespace reset_sub_topic">
+    <gazebo>
+      <plugin name="reset_plugin" filename="libResetPlugin.so">
       </plugin>
     </gazebo>

Commit message: add mavlink_tcp_port for multiple uav simultation

File: models/rotors_description/urdf/component_snippets.xacro (robot description, xacro)
@@ -128,5 +128,5 @@
   </xacro:macro>
   <!-- Macro to add the mavlink interface. -->
-  <xacro:macro name="mavlink_interface_macro" params="namespace imu_sub_topic gps_sub_topic mavlink_addr mavlink_udp_port serial_enabled serial_device baudrate qgc_addr qgc_udp_port hil_mode hil_state_level vehicle_is_tailsitter send_vision_estimation send_odometry enable_lockstep use_tcp">
+  <xacro:macro name="mavlink_interface_macro" params="namespace imu_sub_topic gps_sub_topic mavlink_addr mavlink_udp_port mavlink_tcp_port serial_enabled serial_device baudrate qgc_addr qgc_udp_port hil_mode hil_state_level vehicle_is_tailsitter send_vision_estimation send_odometry enable_lockstep use_tcp">
     <gazebo>
       <plugin name="mavlink_interface" filename="libgazebo_mavlink_interface.so">
@@ -136,4 +136,5 @@
         <mavlink_addr>$(arg mavlink_addr)</mavlink_addr>
         <mavlink_udp_port>$(arg mavlink_udp_port)</mavlink_udp_port>
+        <mavlink_tcp_port>$(arg mavlink_tcp_port)</mavlink_tcp_port>
         <serialEnabled>$(arg serial_enabled)</serialEnabled>
         <serialDevice>$(arg serial_device)</serialDevice>

File: models/rotors_description/urdf/iris_base.xacro (robot description, xacro)
@@ -7,4 +7,5 @@
   <xacro:arg name='mavlink_addr' default='INADDR_ANY' />
   <xacro:arg name='mavlink_udp_port' default='14560' />
+  <xacro:arg name='mavlink_tcp_port' default='4560' />
   <xacro:arg name='serial_enabled' default='false' />
   <xacro:arg name='serial_device' default='/dev/ttyACM0' />
@@ -56,4 +57,5 @@
     mavlink_addr="$(arg mavlink_addr)"
     mavlink_udp_port="$(arg mavlink_udp_port)"
+    mavlink_tcp_port="$(arg mavlink_tcp_port)"
     serial_enabled="$(arg serial_enabled)"
     serial_device="$(arg serial_device)"

Commit message: add magnetometer plugin generation to .xacro

File: models/rotors_description/urdf/component_snippets.xacro (robot description, xacro)
@@ -118,5 +118,5 @@
     </gazebo>
   </xacro:macro>
-    <!-- Macro to add the gps_plugin. -->
+  <!-- Macro to add the gps_plugin. -->
   <xacro:macro name="gps_plugin_macro" params="namespace gps_noise">
     <gazebo>
@@ -127,6 +127,17 @@
     </gazebo>
   </xacro:macro>
+  <!-- Macro to add the magnetometer_plugin. -->
+  <xacro:macro name="magnetometer_plugin_macro" params="namespace pub_rate noise_density mag_topic">
+    <gazebo>
+      <plugin name="magnetometer_plugin" filename="libgazebo_magnetometer_plugin.so">
+        <robotNamespace>${namespace}</robotNamespace>
+        <pubRate>${pub_rate}</pubRate>
+        <noiseDensity>${noise_density}</noiseDensity>
+        <magTopic>${mag_topic}</magTopic>
+      </plugin>
+    </gazebo>
+  </xacro:macro>
   <!-- Macro to add the mavlink interface. -->
-  <xacro:macro name="mavlink_interface_macro" params="namespace imu_sub_topic gps_sub_topic mavlink_addr mavlink_udp_port mavlink_tcp_port serial_enabled serial_device baudrate qgc_addr qgc_udp_port hil_mode hil_state_level vehicle_is_tailsitter send_vision_estimation send_odometry enable_lockstep use_tcp">
+  <xacro:macro name="mavlink_interface_macro" params="namespace imu_sub_topic gps_sub_topic mag_sub_topic mavlink_addr mavlink_udp_port mavlink_tcp_port serial_enabled serial_device baudrate qgc_addr qgc_udp_port hil_mode hil_state_level vehicle_is_tailsitter send_vision_estimation send_odometry enable_lockstep use_tcp">
     <gazebo>
       <plugin name="mavlink_interface" filename="libgazebo_mavlink_interface.so">
@@ -134,4 +145,5 @@
         <imuSubTopic>${imu_sub_topic}</imuSubTopic>
         <gpsSubTopic>${gps_sub_topic}</gpsSubTopic>
+        <magSubTopic>${mag_sub_topic}</magSubTopic>
         <mavlink_addr>$(arg mavlink_addr)</mavlink_addr>
         <mavlink_udp_port>$(arg mavlink_udp_port)</mavlink_udp_port>

File: models/rotors_description/urdf/iris_base.xacro (robot description, xacro)
@@ -43,5 +43,5 @@
         />
   </xacro:if>
-    <!-- Instantiate gps plugin. -->
+  <!-- Instantiate gps plugin. -->
   <xacro:gps_plugin_macro
     namespace="${namespace}"
@@ -49,4 +49,12 @@
     >
   </xacro:gps_plugin_macro>
+  <!-- Instantiate magnetometer plugin. -->
+  <xacro:magnetometer_plugin_macro
+    namespace="${namespace}"
+    pub_rate="20"
+    noise_density="0.01"
+    mag_topic="/mag"
+    >
+  </xacro:magnetometer_plugin_macro>
   <xacro:if value="$(arg enable_mavlink_interface)">
   <!-- Instantiate mavlink telemetry interface. -->
@@ -55,4 +63,5 @@
     imu_sub_topic="/imu"
     gps_sub_topic="/gps"
+    mag_sub_topic="/mag"
     mavlink_addr="$(arg mavlink_addr)"
     mavlink_udp_port="$(arg mavlink_udp_port)"

Commit message: add barometer plugin generation to .xacro

File: models/rotors_description/urdf/component_snippets.xacro (robot description, xacro)
@@ -140,6 +140,16 @@
     </gazebo>
   </xacro:macro>
+  <!-- Macro to add the barometer_plugin. -->
+  <xacro:macro name="barometer_plugin_macro" params="namespace pub_rate baro_topic">
+    <gazebo>
+      <plugin name="barometer_plugin" filename="libgazebo_barometer_plugin.so">
+        <robotNamespace>${namespace}</robotNamespace>
+        <pubRate>${pub_rate}</pubRate>
+        <baroTopic>${baro_topic}</baroTopic>
+      </plugin>
+    </gazebo>
+  </xacro:macro>
   <!-- Macro to add the mavlink interface. -->
-  <xacro:macro name="mavlink_interface_macro" params="namespace imu_sub_topic gps_sub_topic mag_sub_topic mavlink_addr mavlink_udp_port mavlink_tcp_port serial_enabled serial_device baudrate qgc_addr qgc_udp_port hil_mode hil_state_level vehicle_is_tailsitter send_vision_estimation send_odometry enable_lockstep use_tcp">
+  <xacro:macro name="mavlink_interface_macro" params="namespace imu_sub_topic gps_sub_topic mag_sub_topic baro_sub_topic mavlink_addr mavlink_udp_port mavlink_tcp_port serial_enabled serial_device baudrate qgc_addr qgc_udp_port hil_mode hil_state_level vehicle_is_tailsitter send_vision_estimation send_odometry enable_lockstep use_tcp">
     <gazebo>
       <plugin name="mavlink_interface" filename="libgazebo_mavlink_interface.so">
@@ -148,4 +158,5 @@
         <gpsSubTopic>${gps_sub_topic}</gpsSubTopic>
         <magSubTopic>${mag_sub_topic}</magSubTopic>
+        <baroSubTopic>${baro_sub_topic}</baroSubTopic>
         <mavlink_addr>$(arg mavlink_addr)</mavlink_addr>
         <mavlink_udp_port>$(arg mavlink_udp_port)</mavlink_udp_port>

File: models/rotors_description/urdf/iris_base.xacro (robot description, xacro)
@@ -59,4 +59,11 @@
     >
   </xacro:magnetometer_plugin_macro>
+  <!-- Instantiate barometer plugin. -->
+  <xacro:barometer_plugin_macro
+    namespace="${namespace}"
+    pub_rate="10"
+    baro_topic="/baro"
+    >
+  </xacro:barometer_plugin_macro>
   <xacro:if value="$(arg enable_mavlink_interface)">
   <!-- Instantiate mavlink telemetry interface. -->
@@ -66,4 +73,5 @@
     gps_sub_topic="/gps"
     mag_sub_topic="/mag"
+    baro_sub_topic="/baro"
     mavlink_addr="$(arg mavlink_addr)"
     mavlink_udp_port="$(arg mavlink_udp_port)"

Commit message: change default noise model parameters based on ADIS16448 datasheet

File: models/rotors_description/urdf/component_snippets.xacro (robot description, xacro)
@@ -128,5 +128,5 @@
   </xacro:macro>
   <!-- Macro to add the magnetometer_plugin. -->
-  <xacro:macro name="magnetometer_plugin_macro" params="namespace pub_rate noise_density mag_topic">
+  <xacro:macro name="magnetometer_plugin_macro" params="namespace pub_rate noise_density random_walk bias_correlation_time mag_topic">
     <gazebo>
       <plugin name="magnetometer_plugin" filename="libgazebo_magnetometer_plugin.so">
@@ -134,4 +134,6 @@
         <pubRate>${pub_rate}</pubRate>
         <noiseDensity>${noise_density}</noiseDensity>
+        <randomWalk>${random_walk}</randomWalk>
+        <biasCorrelationTime>${bias_correlation_time}</biasCorrelationTime>
         <magTopic>${mag_topic}</magTopic>
       </plugin>

File: models/rotors_description/urdf/iris_base.xacro (robot description, xacro)
@@ -53,5 +53,7 @@
     namespace="${namespace}"
     pub_rate="20"
-    noise_density="0.01"
+    noise_density="0.0004"
+    random_walk="0.0000064"
+    bias_correlation_time="600"
     mag_topic="/mag"
     >
