Commit message: iris allowing multirobot

File: models/rotors_description/urdf/component_snippets.xacro (robot description, xacro)
@@ -24,6 +24,6 @@
         <robotNamespace>${namespace}</robotNamespace>
         <bagFileName>${bag_file}</bagFileName>
-        <linkName>base_link</linkName>
-        <frameId>base_link</frameId>
+        <linkName>${namespace}_base_link</linkName>
+        <frameId>${namespace}_base_link</frameId>
         <commandAttitudeThrustSubTopic>command/attitude</commandAttitudeThrustSubTopic>
         <commandAttitudeThrustPubTopic>command/attitude</commandAttitudeThrustPubTopic>

File: models/rotors_description/urdf/iris.xacro (robot description, xacro)
@@ -2,5 +2,5 @@
 <robot name="iris" xmlns:xacro="http://ros.org/wiki/xacro">
   <!-- Properties -->
-  <xacro:property name="namespace" value="" />
+  <xacro:property name="namespace" value="$(arg name)" />
   <xacro:property name="rotor_velocity_slowdown_sim" value="10" />
   <xacro:property name="mesh_file" value="iris.stl" />
@@ -65,5 +65,5 @@
     motor_constant="${motor_constant}"
     moment_constant="${moment_constant}"
-    parent="base_link"
+    parent="${namespace}_base_link"
     mass_rotor="${mass_rotor}"
     radius_rotor="${radius_rotor}"
@@ -86,5 +86,5 @@
     motor_constant="${motor_constant}"
     moment_constant="${moment_constant}"
-    parent="base_link"
+    parent="${namespace}_base_link"
     mass_rotor="${mass_rotor}"
     radius_rotor="${radius_rotor}"
@@ -106,5 +106,5 @@
     motor_constant="${motor_constant}"
     moment_constant="${moment_constant}"
-    parent="base_link"
+    parent="${namespace}_base_link"
     mass_rotor="${mass_rotor}"
     radius_rotor="${radius_rotor}"
@@ -126,5 +126,5 @@
     motor_constant="${motor_constant}"
     moment_constant="${moment_constant}"
-    parent="base_link"
+    parent="${namespace}_base_link"
     mass_rotor="${mass_rotor}"
     radius_rotor="${radius_rotor}"

File: models/rotors_description/urdf/iris_base.xacro (robot description, xacro)
@@ -100,5 +100,5 @@
     namespace="${namespace}"
     imu_suffix=""
-    parent_link="base_link"
+    parent_link="${namespace}_base_link"
     imu_topic="/imu"
     mass_imu_sensor="0.015"
@@ -120,5 +120,5 @@
       namespace="${namespace}"
       imu_suffix="gt"
-      parent_link="base_link"
+      parent_link="${namespace}_base_link"
       imu_topic="ground_truth/imu"
       mass_imu_sensor="0.00001"
@@ -139,5 +139,5 @@
       namespace="${namespace}/ground_truth"
       odometry_sensor_suffix="gt"
-      parent_link="base_link"
+      parent_link="${namespace}_base_link"
       pose_topic="pose"
       pose_with_covariance_topic="pose_with_covariance"

File: models/rotors_description/urdf/multirotor_base.xacro (robot description, xacro)
@@ -20,11 +20,11 @@
   <xacro:macro name="multirotor_base_macro"
     params="robot_namespace mass body_width body_height mesh_file mesh_scale color *inertia">
-    <link name="base_link"></link>
-    <joint name="base_joint" type="fixed">
+    <link name="${robot_namespace}_base_link"></link>
+    <joint name="${robot_namespace}_base_joint" type="fixed">
       <origin xyz="0 0 0" rpy="0 0 0" />
-      <parent link="base_link" />
-      <child link="base_link_inertia" />
+      <parent link="${robot_namespace}_base_link" />
+      <child link="${robot_namespace}_base_link_inertia" />
     </joint>
-    <link name="base_link_inertia">
+    <link name="${robot_namespace}_base_link_inertia">
       <inertial>
         <mass value="${mass}" />  <!-- [kg] -->
@@ -51,9 +51,9 @@
       <plugin filename="libgazebo_multirotor_base_plugin.so" name="rosbag">
         <robotNamespace>${robot_namespace}</robotNamespace>
-        <linkName>base_link</linkName>
+        <linkName>${robot_namespace}_base_link</linkName>
         <rotorVelocitySlowdownSim>${rotor_velocity_slowdown_sim}</rotorVelocitySlowdownSim>
       </plugin>
     </gazebo>
-    <gazebo reference="base_link">
+    <gazebo reference="${robot_namespace}_base_link">
       <material>Gazebo/${color}</material>
       <collision name='base_link_inertia_collision'>
@@ -75,5 +75,5 @@
   <xacro:macro name="vertical_rotor"
     params="robot_namespace suffix direction motor_constant moment_constant parent mass_rotor radius_rotor time_constant_up time_constant_down max_rot_velocity motor_number rotor_drag_coefficient rolling_moment_coefficient color mesh mesh_scale *origin *inertia">
-    <joint name="rotor_${motor_number}_joint" type="continuous">
+    <joint name="${robot_namespace}_rotor_${motor_number}_joint" type="continuous">
       <xacro:insert_block name="origin" />
       <axis xyz="0 0 1" />
@@ -81,10 +81,10 @@
       <!-- <limit effort="2000" velocity="${max_rot_velocity}" /> -->
       <parent link="${parent}" />
-      <child link="rotor_${motor_number}" />
+      <child link="${robot_namespace}_rotor_${motor_number}" />
     </joint>
     <!-- TODO(ff): not currently set because it's not yet supported -->
     <!-- <gazebo reference="rotor_${motor_number}_joint"> <axis> <xyz>0 0 1</xyz>
       <limit> <velocity> ${max_rot_velocity} </velocity> </limit> </axis> </gazebo> -->
-    <link name="rotor_${motor_number}">
+    <link name="${robot_namespace}_rotor_${motor_number}">
       <inertial>
         <mass value="${mass_rotor}" /> <!-- [kg] -->
@@ -109,6 +109,6 @@
       <plugin name="${suffix}_motor_model" filename="libgazebo_motor_model.so">
         <robotNamespace>${robot_namespace}</robotNamespace>
-        <jointName>rotor_${motor_number}_joint</jointName>
-        <linkName>rotor_${motor_number}</linkName>
+        <jointName>${robot_namespace}_rotor_${motor_number}_joint</jointName>
+        <linkName>${robot_namespace}_rotor_${motor_number}</linkName>
         <turningDirection>${direction}</turningDirection>
         <timeConstantUp>${time_constant_up}</timeConstantUp>
@@ -136,5 +136,5 @@
       </plugin>
     </gazebo>
-    <gazebo reference="rotor_${motor_number}">
+    <gazebo reference="${robot_namespace}_rotor_${motor_number}">
       <material>Gazebo/${color}</material>
     </gazebo>

Commit message: iris including fpv camera

File: models/rotors_description/urdf/component_snippets.xacro (robot description, xacro)
@@ -32,4 +32,84 @@
     </gazebo>
   </xacro:macro>
+  <xacro:arg name='camera_udp_port' default='5600' />
+  <xacro:macro name="fpv_cam">
+    <link name='camera_link'>
+      <pose rpy="0  0  0" xyz="0  0  0"/>
+      <inertial>
+        <mass value="0.015"/>
+        <origin rpy="0  0  0" xyz="0  0  0"/>
+        <inertia ixx="4.15e-6" ixy="0" ixz="0" iyy="2.407e-6" iyz="0" izz="2.407e-6"/>
+      </inertial>
+      <collision name="camera_link_inertia_collision">
+        <origin rpy="0  0  0" xyz="0  0  0"/>
+        <geometry>
+          <box size="0.01 0.01 0.01"/>
+        </geometry>
+      </collision>
+      <visual name="camera_link_inertia_visual">
+        <origin rpy="0  0  0" xyz="0  0  0"/>
+        <geometry>
+          <box size="0.01 0.01 0.01"/>
+        </geometry>
+      </visual>
+    </link>
+    <gazebo reference="camera_link">
+      <self_collide>0</self_collide>
+      <kinematic>0</kinematic>
+      <sensor name='camera' type='camera'>
+        <camera name='__default__'>
+          <horizontal_fov>1.047</horizontal_fov>
+          <image>
+            <width>320</width>
+            <height>240</height>
+          </image>
+          <clip>
+            <near>0.1</near>
+            <far>15000</far>
+          </clip>
+          <lens>
+            <type>custom</type>
+            <custom_function>
+              <c1>1.05</c1>
+              <c2>4</c2>
+              <f>1</f>
+              <fun>tan</fun>
+            </custom_function>
+            <scale_to_hfov>1</scale_to_hfov>
+            <cutoff_angle>3.1415</cutoff_angle>
+            <env_texture_size>1080</env_texture_size>
+          </lens>
+        </camera>
+        <always_on>1</always_on>
+        <update_rate>30</update_rate>
+        <visualize>1</visualize>
+        <plugin name='camera_plugin' filename='libgazebo_ros_camera.so'>
+            <robotNamespace></robotNamespace>
+          <alwaysOn>true</alwaysOn>
+          <imageTopicName>image_raw</imageTopicName>
+          <cameraInfoTopicName>camera_info</cameraInfoTopicName>
+          <updateRate>30.0</updateRate>
+          <cameraName>usb_cam</cameraName>
+          <frameName>/robot_camera_link</frameName>
+          <CxPrime>320.5</CxPrime>
+          <Cx>320.5</Cx>
+          <Cy>240.5</Cy>
+          <hackBaseline>0</hackBaseline>
+          <focalLength>277.191356</focalLength>
+          <distortionK1>0.0</distortionK1>
+          <distortionK2>0.0</distortionK2>
+          <distortionK3>0.0</distortionK3>
+          <distortionT1>0.0</distortionT1>
+          <distortionT2>0.0</distortionT2>
+        </plugin>
+        <!-- GStreamer camera plugin (needs a lot of CPU! Consider lowering the
+           camera image size) -->
+        <plugin name="GstCameraPlugin" filename="libgazebo_gst_camera_plugin.so">
+          <robotNamespace></robotNamespace>
+          <udpPort>$(arg camera_udp_port)</udpPort>
+        </plugin>
+      </sensor>
+    </gazebo>
+    </xacro:macro>
   <!-- Macro to add a camera. -->
   <xacro:macro name="camera_macro"
@@ -583,3 +663,13 @@
     </xacro:imu_plugin_macro>
   </xacro:macro>
+  <xacro:if value="$(arg enable_camera)">
+    <xacro:fpv_cam/>
+    <joint name="fpv_joint" type="fixed">
+      <parent link="$(arg name)_base_link"/>
+      <child link="camera_link"/>
+      <origin rpy="0  0  0" xyz="0  0  0"/>
+      <axis xyz="0  0  1"/>
+      <limit effort="0.0" lower="0.0" upper="0.0" velocity="0.0"/>
+    </joint>
+  </xacro:if>
 </robot>

File: models/rotors_description/urdf/iris_base.xacro (robot description, xacro)
@@ -29,4 +29,5 @@
   <xacro:arg name='enable_ground_truth' default='false' />
   <xacro:arg name='enable_logging' default='false' />
+  <xacro:arg name='enable_camera' default='false' />
   <xacro:arg name='log_file' default='iris' />
   <!-- macros for gazebo plugins, sensors -->

Commit message: Iris including joint_state_publisher

File: models/rotors_description/urdf/component_snippets.xacro (robot description, xacro)
@@ -112,4 +112,18 @@
     </gazebo>
     </xacro:macro>
+  <xacro:macro name="joint_state_publisher_macro"
+    params="namespace">
+    <gazebo>
+      <plugin name="joint_state_publisher" filename="libgazebo_ros_joint_state_publisher.so">
+        <joint_name>${namespace}::${namespace}/imugt_link</joint_name>
+        <joint_name>${namespace}::${namespace}/ground_truth/odometry_sensorgt_link</joint_name>
+        <joint_name>${namespace}::${namespace}_rotor_0_joint</joint_name>
+        <joint_name>${namespace}::${namespace}_rotor_1_joint</joint_name>
+        <joint_name>${namespace}::${namespace}_rotor_2_joint</joint_name>
+        <joint_name>${namespace}::${namespace}_rotor_3_joint</joint_name>
+      <update_rate>100</update_rate>
+      </plugin>
+    </gazebo>
+  </xacro:macro>
   <!-- Macro to add a camera. -->
   <xacro:macro name="camera_macro"
@@ -673,3 +687,6 @@
     </joint>
   </xacro:if>
+  <xacro:joint_state_publisher_macro
+    namespace="$(arg name)" >
+  </xacro:joint_state_publisher_macro>
 </robot>

Commit message: Add xacro files for plane model

File: models/rotors_description/urdf/component_snippets.xacro (robot description, xacro)
@@ -273,4 +273,81 @@
             <zero_position_armed>0</zero_position_armed>
             <joint_control_type>position</joint_control_type>
+          </channel>
+        </control_channels>
+      </plugin>
+    </gazebo>
+  </xacro:macro>
+  <!-- Macro to add the mavlink interface for a fixed-wing model. -->
+  <xacro:macro name="mavlink_interface_macro_fw" params="namespace imu_sub_topic gps_sub_topic mag_sub_topic baro_sub_topic mavlink_addr mavlink_udp_port mavlink_tcp_port serial_enabled serial_device baudrate qgc_addr qgc_udp_port sdk_addr sdk_udp_port hil_mode hil_state_level vehicle_is_tailsitter send_vision_estimation send_odometry enable_lockstep use_tcp">
+    <gazebo>
+      <plugin name="mavlink_interface" filename="libgazebo_mavlink_interface.so">
+        <robotNamespace>${namespace}</robotNamespace>
+        <imuSubTopic>${imu_sub_topic}</imuSubTopic>
+        <gpsSubTopic>${gps_sub_topic}</gpsSubTopic>
+        <magSubTopic>${mag_sub_topic}</magSubTopic>
+        <baroSubTopic>${baro_sub_topic}</baroSubTopic>
+        <mavlink_addr>$(arg mavlink_addr)</mavlink_addr>
+        <mavlink_udp_port>$(arg mavlink_udp_port)</mavlink_udp_port>
+        <mavlink_tcp_port>$(arg mavlink_tcp_port)</mavlink_tcp_port>
+        <serialEnabled>$(arg serial_enabled)</serialEnabled>
+        <serialDevice>$(arg serial_device)</serialDevice>
+        <baudRate>$(arg baudrate)</baudRate>
+        <qgc_addr>$(arg qgc_addr)</qgc_addr>
+        <qgc_udp_port>$(arg qgc_udp_port)</qgc_udp_port>
+        <sdk_addr>$(arg sdk_addr)</sdk_addr>
+        <sdk_udp_port>$(arg sdk_udp_port)</sdk_udp_port>
+        <hil_mode>$(arg hil_mode)</hil_mode>
+        <hil_state_level>$(arg hil_state_level)</hil_state_level>
+        <vehicle_is_tailsitter>$(arg vehicle_is_tailsitter)</vehicle_is_tailsitter>
+        <send_vision_estimation>$(arg send_vision_estimation)</send_vision_estimation>
+        <send_odometry>$(arg send_odometry)</send_odometry>
+        <enable_lockstep>$(arg enable_lockstep)</enable_lockstep>
+        <use_tcp>$(arg use_tcp)</use_tcp>
+        <motorSpeedCommandPubTopic>/gazebo/command/motor_speed</motorSpeedCommandPubTopic>
+        <control_channels>
+          <channel name="rudder">
+            <input_index>2</input_index>
+            <input_offset>0</input_offset>
+            <input_scaling>1</input_scaling>
+            <zero_position_disarmed>0</zero_position_disarmed>
+            <zero_position_armed>0</zero_position_armed>
+            <joint_control_type>position_kinematic</joint_control_type>
+            <joint_name>rudder_joint</joint_name>
+          </channel>
+          <channel name="rotor_4">
+            <input_index>4</input_index>
+            <input_offset>0</input_offset>
+            <input_scaling>3500</input_scaling>
+            <zero_position_disarmed>0</zero_position_disarmed>
+            <zero_position_armed>0</zero_position_armed>
+            <joint_control_type>velocity</joint_control_type>
+            <joint_name>rotor_4_joint</joint_name>
+          </channel>
+          <channel name="left_aileron">
+            <input_index>5</input_index>
+            <input_offset>0</input_offset>
+            <input_scaling>1</input_scaling>
+            <zero_position_disarmed>0</zero_position_disarmed>
+            <zero_position_armed>0</zero_position_armed>
+            <joint_control_type>position_kinematic</joint_control_type>
+            <joint_name>left_elevon_joint</joint_name>
+          </channel>
+          <channel name="right_aileron">
+            <input_index>6</input_index>
+            <input_offset>0</input_offset>
+            <input_scaling>1</input_scaling>
+            <zero_position_disarmed>0</zero_position_disarmed>
+            <zero_position_armed>0</zero_position_armed>
+            <joint_control_type>position_kinematic</joint_control_type>
+            <joint_name>right_elevon_joint</joint_name>
+          </channel>
+          <channel name="elevator">
+            <input_index>7</input_index>
+            <input_offset>0</input_offset>
+            <input_scaling>1</input_scaling>
+            <zero_position_disarmed>0</zero_position_disarmed>
+            <zero_position_armed>0</zero_position_armed>
+            <joint_control_type>position_kinematic</joint_control_type>
+            <joint_name>elevator_joint</joint_name>
           </channel>
         </control_channels>
