Commit message: add GPS model to xacro-generated models, update licenses; gazebo_mavlink_interface: use joint names for subscription generation

File: models/rotors_description/urdf/component_snippets.xacro (robot description, xacro)
@@ -6,4 +6,5 @@
   Copyright 2015 Janosch Nikolic, ASL, ETH Zurich, Switzerland
   Copyright 2015 Markus Achtelik, ASL, ETH Zurich, Switzerland
+  Copyright 2015-2020 PX4 Development Team. All rights reserved.
   Licensed under the Apache License, Version 2.0 (the "License");
   you may not use this file except in compliance with the License.
@@ -17,4 +18,51 @@
 -->
 <robot xmlns:xacro="http://ros.org/wiki/xacro">
+  <!-- Macro to a add a GPS sensor. -->
+  <xacro:macro name="gps_macro"
+    params="gps_name pos_x pos_y pos_z gps_noise namespace parent_link">
+    <gazebo>
+      <model name="${gps_name}">
+        <link name="link">
+          <pose>${pos_x} ${pos_y} ${pos_z} 0 0 0</pose>
+          <inertial>
+            <pose>0 0 0 0 0 0</pose>
+            <mass>0.01</mass>
+            <inertia>
+              <ixx>2.1733e-6</ixx>
+              <ixy>0</ixy>
+              <ixz>0</ixz>
+              <iyy>2.1733e-6</iyy>
+              <iyz>0</iyz>
+              <izz>1.8e-7</izz>
+            </inertia>
+          </inertial>
+          <visual name="visual">
+            <geometry>
+              <cylinder>
+                <radius>0.01</radius>
+                <length>0.002</length>
+              </cylinder>
+            </geometry>
+            <material>
+              <script>
+                <name>Gazebo/Black</name>
+              </script>
+            </material>
+          </visual>
+          <sensor name="gps" type="gps">
+            <pose>0 0 0 0 0 0</pose>
+            <plugin name="gps_plugin" filename="libgazebo_gps_plugin.so">
+              <robotNamespace>${namespace}</robotNamespace>
+              <gpsNoise>${gps_noise}</gpsNoise>
+            </plugin>
+          </sensor>
+        </link>
+      </model>
+      <joint name="gps_joint" type="fixed">
+        <parent>${parent_link}</parent>
+        <child>gps::link</child>
+      </joint>
+    </gazebo>
+  </xacro:macro>
   <!-- Macro to add logging to a bag file. -->
   <xacro:macro name="bag_plugin_macro"
@@ -118,13 +166,4 @@
     </gazebo>
   </xacro:macro>
-  <!-- Macro to add the gps_plugin. -->
-  <xacro:macro name="gps_plugin_macro" params="namespace gps_noise">
-    <gazebo>
-      <plugin name="gps_plugin" filename="libgazebo_gps_plugin.so">
-        <robotNamespace>${namespace}</robotNamespace>
-        <gpsNoise>${gps_noise}</gpsNoise>
-      </plugin>
-    </gazebo>
-  </xacro:macro>
   <!-- Macro to add the magnetometer_plugin. -->
   <xacro:macro name="magnetometer_plugin_macro" params="namespace pub_rate noise_density random_walk bias_correlation_time mag_topic">
@@ -151,10 +190,9 @@
   </xacro:macro>
   <!-- Macro to add the mavlink interface. -->
-  <xacro:macro name="mavlink_interface_macro" params="namespace imu_sub_topic gps_sub_topic mag_sub_topic baro_sub_topic mavlink_addr mavlink_udp_port mavlink_tcp_port serial_enabled serial_device baudrate qgc_addr qgc_udp_port sdk_addr sdk_udp_port hil_mode hil_state_level vehicle_is_tailsitter send_vision_estimation send_odometry enable_lockstep use_tcp">
+  <xacro:macro name="mavlink_interface_macro" params="namespace imu_sub_topic mag_sub_topic baro_sub_topic mavlink_addr mavlink_udp_port mavlink_tcp_port serial_enabled serial_device baudrate qgc_addr qgc_udp_port sdk_addr sdk_udp_port hil_mode hil_state_level vehicle_is_tailsitter send_vision_estimation send_odometry enable_lockstep use_tcp">
     <gazebo>
       <plugin name="mavlink_interface" filename="libgazebo_mavlink_interface.so">
         <robotNamespace>${namespace}</robotNamespace>
         <imuSubTopic>${imu_sub_topic}</imuSubTopic>
-        <gpsSubTopic>${gps_sub_topic}</gpsSubTopic>
         <magSubTopic>${mag_sub_topic}</magSubTopic>
         <baroSubTopic>${baro_sub_topic}</baroSubTopic>
@@ -279,10 +317,9 @@
   </xacro:macro>
   <!-- Macro to add the mavlink interface for a fixed-wing model. -->
-  <xacro:macro name="mavlink_interface_macro_fw" params="namespace imu_sub_topic gps_sub_topic mag_sub_topic baro_sub_topic mavlink_addr mavlink_udp_port mavlink_tcp_port serial_enabled serial_device baudrate qgc_addr qgc_udp_port sdk_addr sdk_udp_port hil_mode hil_state_level vehicle_is_tailsitter send_vision_estimation send_odometry enable_lockstep use_tcp">
+  <xacro:macro name="mavlink_interface_macro_fw" params="namespace imu_sub_topic mag_sub_topic baro_sub_topic mavlink_addr mavlink_udp_port mavlink_tcp_port serial_enabled serial_device baudrate qgc_addr qgc_udp_port sdk_addr sdk_udp_port hil_mode hil_state_level vehicle_is_tailsitter send_vision_estimation send_odometry enable_lockstep use_tcp">
     <gazebo>
       <plugin name="mavlink_interface" filename="libgazebo_mavlink_interface.so">
         <robotNamespace>${namespace}</robotNamespace>
         <imuSubTopic>${imu_sub_topic}</imuSubTopic>
-        <gpsSubTopic>${gps_sub_topic}</gpsSubTopic>
         <magSubTopic>${mag_sub_topic}</magSubTopic>
         <baroSubTopic>${baro_sub_topic}</baroSubTopic>
@@ -356,10 +393,9 @@
   </xacro:macro>
   <!-- Macro to add the mavlink interface for a fixed-wing model. -->
-  <xacro:macro name="mavlink_interface_macro_vtol" params="namespace imu_sub_topic gps_sub_topic mag_sub_topic baro_sub_topic mavlink_addr mavlink_udp_port mavlink_tcp_port serial_enabled serial_device baudrate qgc_addr qgc_udp_port sdk_addr sdk_udp_port hil_mode hil_state_level vehicle_is_tailsitter send_vision_estimation send_odometry enable_lockstep use_tcp">
+  <xacro:macro name="mavlink_interface_macro_vtol" params="namespace imu_sub_topic mag_sub_topic baro_sub_topic mavlink_addr mavlink_udp_port mavlink_tcp_port serial_enabled serial_device baudrate qgc_addr qgc_udp_port sdk_addr sdk_udp_port hil_mode hil_state_level vehicle_is_tailsitter send_vision_estimation send_odometry enable_lockstep use_tcp">
     <gazebo>
       <plugin name='mavlink_interface' filename='libgazebo_mavlink_interface.so'>
         <robotNamespace>${namespace}</robotNamespace>
         <imuSubTopic>${imu_sub_topic}</imuSubTopic>
-        <gpsSubTopic>${gps_sub_topic}</gpsSubTopic>
         <magSubTopic>${mag_sub_topic}</magSubTopic>
         <baroSubTopic>${baro_sub_topic}</baroSubTopic>

File: models/rotors_description/urdf/fixedwing_base.xacro (robot description, xacro)
@@ -6,4 +6,5 @@
   Copyright 2015 Janosch Nikolic, ASL, ETH Zurich, Switzerland
   Copyright 2015 Markus Achtelik, ASL, ETH Zurich, Switzerland
+  Copyright 2020 PX4 Development Team. All rights reserved.
   Licensed under the Apache License, Version 2.0 (the "License");
   you may not use this file except in compliance with the License.

File: models/rotors_description/urdf/iris.xacro (robot description, xacro)
@@ -1,3 +1,34 @@
 <?xml version="1.0"?>
+<!--
+  -   Copyright (c) 2015-2020 PX4 Development Team. All rights reserved.
+  -
+  - Redistribution and use in source and binary forms, with or without
+  - modification, are permitted provided that the following conditions
+  - are met:
+  -
+  - 1. Redistributions of source code must retain the above copyright
+  -    notice, this list of conditions and the following disclaimer.
+  - 2. Redistributions in binary form must reproduce the above copyright
+  -    notice, this list of conditions and the following disclaimer in
+  -    the documentation and/or other materials provided with the
+  -    distribution.
+  - 3. Neither the name PX4 nor the names of its contributors may be
+  -    used to endorse or promote products derived from this software
+  -    without specific prior written permission.
+  -
+  - THIS SOFTWARE IS PROVIDED BY THE COPYRIGHT HOLDERS AND CONTRIBUTORS
+  - "AS IS" AND ANY EXPRESS OR IMPLIED WARRANTIES, INCLUDING, BUT NOT
+  - LIMITED TO, THE IMPLIED WARRANTIES OF MERCHANTABILITY AND FITNESS
+  - FOR A PARTICULAR PURPOSE ARE DISCLAIMED. IN NO EVENT SHALL THE
+  - COPYRIGHT OWNER OR CONTRIBUTORS BE LIABLE FOR ANY DIRECT, INDIRECT,
+  - INCIDENTAL, SPECIAL, EXEMPLARY, OR CONSEQUENTIAL DAMAGES (INCLUDING,
+  - BUT NOT LIMITED TO, PROCUREMENT OF SUBSTITUTE GOODS OR SERVICES; LOSS
+  - OF USE, DATA, OR PROFITS; OR BUSINESS INTERRUPTION) HOWEVER CAUSED
+  - AND ON ANY THEORY OF LIABILITY, WHETHER IN CONTRACT, STRICT
+  - LIABILITY, OR TORT (INCLUDING NEGLIGENCE OR OTHERWISE) ARISING IN
+  - ANY WAY OUT OF THE USE OF THIS SOFTWARE, EVEN IF ADVISED OF THE
+  - POSSIBILITY OF SUCH DAMAGE.
+  -
+  -->
 <robot name="iris" xmlns:xacro="http://ros.org/wiki/xacro">
   <!-- Properties -->

File: models/rotors_description/urdf/iris_base.xacro (robot description, xacro)
@@ -1,3 +1,34 @@
 <?xml version="1.0"?>
+<!--
+  -   Copyright (c) 2015-2020 PX4 Development Team. All rights reserved.
+  -
+  - Redistribution and use in source and binary forms, with or without
+  - modification, are permitted provided that the following conditions
+  - are met:
+  -
+  - 1. Redistributions of source code must retain the above copyright
+  -    notice, this list of conditions and the following disclaimer.
+  - 2. Redistributions in binary form must reproduce the above copyright
+  -    notice, this list of conditions and the following disclaimer in
+  -    the documentation and/or other materials provided with the
+  -    distribution.
+  - 3. Neither the name PX4 nor the names of its contributors may be
+  -    used to endorse or promote products derived from this software
+  -    without specific prior written permission.
+  -
+  - THIS SOFTWARE IS PROVIDED BY THE COPYRIGHT HOLDERS AND CONTRIBUTORS
+  - "AS IS" AND ANY EXPRESS OR IMPLIED WARRANTIES, INCLUDING, BUT NOT
+  - LIMITED TO, THE IMPLIED WARRANTIES OF MERCHANTABILITY AND FITNESS
+  - FOR A PARTICULAR PURPOSE ARE DISCLAIMED. IN NO EVENT SHALL THE
+  - COPYRIGHT OWNER OR CONTRIBUTORS BE LIABLE FOR ANY DIRECT, INDIRECT,
+  - INCIDENTAL, SPECIAL, EXEMPLARY, OR CONSEQUENTIAL DAMAGES (INCLUDING,
+  - BUT NOT LIMITED TO, PROCUREMENT OF SUBSTITUTE GOODS OR SERVICES; LOSS
+  - OF USE, DATA, OR PROFITS; OR BUSINESS INTERRUPTION) HOWEVER CAUSED
+  - AND ON ANY THEORY OF LIABILITY, WHETHER IN CONTRACT, STRICT
+  - LIABILITY, OR TORT (INCLUDING NEGLIGENCE OR OTHERWISE) ARISING IN
+  - ANY WAY OUT OF THE USE OF THIS SOFTWARE, EVEN IF ADVISED OF THE
+  - POSSIBILITY OF SUCH DAMAGE.
+  -
+  -->
 <robot name="iris" xmlns:xacro="http://ros.org/wiki/xacro">
   <!-- Properties that can be assigned at build time as arguments.
@@ -45,10 +76,14 @@
         />
   </xacro:if>
-  <!-- Instantiate gps plugin. -->
-  <xacro:gps_plugin_macro
-    namespace="${namespace}"
+  <!-- Mount a GPS module. -->
+  <xacro:gps_macro
+    gps_name="gps"
+    pos_x="0.015"
+    pos_y="0.0"
+    pos_z="0.0"
     gps_noise="true"
-    >
-  </xacro:gps_plugin_macro>
+    namespace=""
+    parent_link="base_link">
+  </xacro:gps_macro>
   <!-- Instantiate magnetometer plugin. -->
   <xacro:magnetometer_plugin_macro
@@ -73,5 +108,4 @@
     namespace="${namespace}"
     imu_sub_topic="/imu"
-    gps_sub_topic="/gps"
     mag_sub_topic="/mag"
     baro_sub_topic="/baro"

File: models/rotors_description/urdf/plane.xacro (robot description, xacro)
@@ -1,3 +1,34 @@
 <?xml version="1.0"?>
+<!--
+  -   Copyright (c) 2020 PX4 Development Team. All rights reserved.
+  -
+  - Redistribution and use in source and binary forms, with or without
+  - modification, are permitted provided that the following conditions
+  - are met:
+  -
+  - 1. Redistributions of source code must retain the above copyright
+  -    notice, this list of conditions and the following disclaimer.
+  - 2. Redistributions in binary form must reproduce the above copyright
+  -    notice, this list of conditions and the following disclaimer in
+  -    the documentation and/or other materials provided with the
+  -    distribution.
+  - 3. Neither the name PX4 nor the names of its contributors may be
+  -    used to endorse or promote products derived from this software
+  -    without specific prior written permission.
+  -
+  - THIS SOFTWARE IS PROVIDED BY THE COPYRIGHT HOLDERS AND CONTRIBUTORS
+  - "AS IS" AND ANY EXPRESS OR IMPLIED WARRANTIES, INCLUDING, BUT NOT
+  - LIMITED TO, THE IMPLIED WARRANTIES OF MERCHANTABILITY AND FITNESS
+  - FOR A PARTICULAR PURPOSE ARE DISCLAIMED. IN NO EVENT SHALL THE
+  - COPYRIGHT OWNER OR CONTRIBUTORS BE LIABLE FOR ANY DIRECT, INDIRECT,
+  - INCIDENTAL, SPECIAL, EXEMPLARY, OR CONSEQUENTIAL DAMAGES (INCLUDING,
+  - BUT NOT LIMITED TO, PROCUREMENT OF SUBSTITUTE GOODS OR SERVICES; LOSS
+  - OF USE, DATA, OR PROFITS; OR BUSINESS INTERRUPTION) HOWEVER CAUSED
+  - AND ON ANY THEORY OF LIABILITY, WHETHER IN CONTRACT, STRICT
+  - LIABILITY, OR TORT (INCLUDING NEGLIGENCE OR OTHERWISE) ARISING IN
+  - ANY WAY OUT OF THE USE OF THIS SOFTWARE, EVEN IF ADVISED OF THE
+  - POSSIBILITY OF SUCH DAMAGE.
+  -
+  -->
 <robot name="plane" xmlns:xacro="http://ros.org/wiki/xacro">
   <!-- Properties -->

File: models/rotors_description/urdf/plane_base.xacro (robot description, xacro)
@@ -1,3 +1,34 @@
 <?xml version="1.0"?>
+<!--
+  -   Copyright (c) 2020 PX4 Development Team. All rights reserved.
+  -
+  - Redistribution and use in source and binary forms, with or without
+  - modification, are permitted provided that the following conditions
+  - are met:
+  -
+  - 1. Redistributions of source code must retain the above copyright
+  -    notice, this list of conditions and the following disclaimer.
+  - 2. Redistributions in binary form must reproduce the above copyright
+  -    notice, this list of conditions and the following disclaimer in
+  -    the documentation and/or other materials provided with the
+  -    distribution.
+  - 3. Neither the name PX4 nor the names of its contributors may be
+  -    used to endorse or promote products derived from this software
+  -    without specific prior written permission.
+  -
+  - THIS SOFTWARE IS PROVIDED BY THE COPYRIGHT HOLDERS AND CONTRIBUTORS
+  - "AS IS" AND ANY EXPRESS OR IMPLIED WARRANTIES, INCLUDING, BUT NOT
+  - LIMITED TO, THE IMPLIED WARRANTIES OF MERCHANTABILITY AND FITNESS
+  - FOR A PARTICULAR PURPOSE ARE DISCLAIMED. IN NO EVENT SHALL THE
+  - COPYRIGHT OWNER OR CONTRIBUTORS BE LIABLE FOR ANY DIRECT, INDIRECT,
+  - INCIDENTAL, SPECIAL, EXEMPLARY, OR CONSEQUENTIAL DAMAGES (INCLUDING,
+  - BUT NOT LIMITED TO, PROCUREMENT OF SUBSTITUTE GOODS OR SERVICES; LOSS
+  - OF USE, DATA, OR PROFITS; OR BUSINESS INTERRUPTION) HOWEVER CAUSED
+  - AND ON ANY THEORY OF LIABILITY, WHETHER IN CONTRACT, STRICT
+  - LIABILITY, OR TORT (INCLUDING NEGLIGENCE OR OTHERWISE) ARISING IN
+  - ANY WAY OUT OF THE USE OF THIS SOFTWARE, EVEN IF ADVISED OF THE
+  - POSSIBILITY OF SUCH DAMAGE.
+  -
+  -->
 <robot name="plane" xmlns:xacro="http://ros.org/wiki/xacro">
   <!-- Properties that can be assigned at build time as arguments.
@@ -45,10 +76,7 @@
         />
   </xacro:if>
-  <!-- Instantiate gps plugin. -->
-  <xacro:gps_plugin_macro
-    namespace="${namespace}"
-    gps_noise="true"
-    >
-  </xacro:gps_plugin_macro>
+  <!-- Mount a GPS module. -->
+  <xacro:gps_macro parent_link="base_link">
+  </xacro:gps_macro>
   <!-- Instantiate magnetometer plugin. -->
   <xacro:magnetometer_plugin_macro
@@ -73,5 +101,4 @@
     namespace="${namespace}"
     imu_sub_topic="/imu"
-    gps_sub_topic="/gps"
     mag_sub_topic="/mag"
     baro_sub_topic="/baro"

File: models/rotors_description/urdf/standard_vtol.xacro (robot description, xacro)
@@ -1,3 +1,34 @@
 <?xml version="1.0"?>
+<!--
+  -   Copyright (c) 2020 PX4 Development Team. All rights reserved.
+  -
+  - Redistribution and use in source and binary forms, with or without
+  - modification, are permitted provided that the following conditions
+  - are met:
+  -
+  - 1. Redistributions of source code must retain the above copyright
+  -    notice, this list of conditions and the following disclaimer.
+  - 2. Redistributions in binary form must reproduce the above copyright
+  -    notice, this list of conditions and the following disclaimer in
+  -    the documentation and/or other materials provided with the
+  -    distribution.
+  - 3. Neither the name PX4 nor the names of its contributors may be
+  -    used to endorse or promote products derived from this software
+  -    without specific prior written permission.
+  -
+  - THIS SOFTWARE IS PROVIDED BY THE COPYRIGHT HOLDERS AND CONTRIBUTORS
+  - "AS IS" AND ANY EXPRESS OR IMPLIED WARRANTIES, INCLUDING, BUT NOT
+  - LIMITED TO, THE IMPLIED WARRANTIES OF MERCHANTABILITY AND FITNESS
+  - FOR A PARTICULAR PURPOSE ARE DISCLAIMED. IN NO EVENT SHALL THE
+  - COPYRIGHT OWNER OR CONTRIBUTORS BE LIABLE FOR ANY DIRECT, INDIRECT,
+  - INCIDENTAL, SPECIAL, EXEMPLARY, OR CONSEQUENTIAL DAMAGES (INCLUDING,
+  - BUT NOT LIMITED TO, PROCUREMENT OF SUBSTITUTE GOODS OR SERVICES; LOSS
+  - OF USE, DATA, OR PROFITS; OR BUSINESS INTERRUPTION) HOWEVER CAUSED
+  - AND ON ANY THEORY OF LIABILITY, WHETHER IN CONTRACT, STRICT
+  - LIABILITY, OR TORT (INCLUDING NEGLIGENCE OR OTHERWISE) ARISING IN
+  - ANY WAY OUT OF THE USE OF THIS SOFTWARE, EVEN IF ADVISED OF THE
+  - POSSIBILITY OF SUCH DAMAGE.
+  -
+  -->
 <robot name="standard_vtol" xmlns:xacro="http://ros.org/wiki/xacro">
   <!-- Properties -->

File: models/rotors_description/urdf/standard_vtol_base.xacro (robot description, xacro)
@@ -1,3 +1,34 @@
 <?xml version="1.0"?>
+<!--
+  -   Copyright (c) 2020 PX4 Development Team. All rights reserved.
+  -
+  - Redistribution and use in source and binary forms, with or without
+  - modification, are permitted provided that the following conditions
+  - are met:
+  -
+  - 1. Redistributions of source code must retain the above copyright
+  -    notice, this list of conditions and the following disclaimer.
+  - 2. Redistributions in binary form must reproduce the above copyright
+  -    notice, this list of conditions and the following disclaimer in
+  -    the documentation and/or other materials provided with the
+  -    distribution.
+  - 3. Neither the name PX4 nor the names of its contributors may be
+  -    used to endorse or promote products derived from this software
+  -    without specific prior written permission.
+  -
+  - THIS SOFTWARE IS PROVIDED BY THE COPYRIGHT HOLDERS AND CONTRIBUTORS
+  - "AS IS" AND ANY EXPRESS OR IMPLIED WARRANTIES, INCLUDING, BUT NOT
+  - LIMITED TO, THE IMPLIED WARRANTIES OF MERCHANTABILITY AND FITNESS
+  - FOR A PARTICULAR PURPOSE ARE DISCLAIMED. IN NO EVENT SHALL THE
+  - COPYRIGHT OWNER OR CONTRIBUTORS BE LIABLE FOR ANY DIRECT, INDIRECT,
+  - INCIDENTAL, SPECIAL, EXEMPLARY, OR CONSEQUENTIAL DAMAGES (INCLUDING,
+  - BUT NOT LIMITED TO, PROCUREMENT OF SUBSTITUTE GOODS OR SERVICES; LOSS
+  - OF USE, DATA, OR PROFITS; OR BUSINESS INTERRUPTION) HOWEVER CAUSED
+  - AND ON ANY THEORY OF LIABILITY, WHETHER IN CONTRACT, STRICT
+  - LIABILITY, OR TORT (INCLUDING NEGLIGENCE OR OTHERWISE) ARISING IN
+  - ANY WAY OUT OF THE USE OF THIS SOFTWARE, EVEN IF ADVISED OF THE
+  - POSSIBILITY OF SUCH DAMAGE.
+  -
+  -->
 <robot name="standard_vtol" xmlns:xacro="http://ros.org/wiki/xacro">
   <!-- Properties that can be assigned at build time as arguments.
@@ -45,10 +76,7 @@
         />
   </xacro:if>
-  <!-- Instantiate gps plugin. -->
-  <xacro:gps_plugin_macro
-    namespace="${namespace}"
-    gps_noise="true"
-    >
-  </xacro:gps_plugin_macro>
+  <!-- Mount a GPS module. -->
+  <xacro:gps_macro parent_link="base_link">
+  </xacro:gps_macro>
   <!-- Instantiate magnetometer plugin. -->
   <xacro:magnetometer_plugin_macro
@@ -73,5 +101,4 @@
     namespace="${namespace}"
     imu_sub_topic="/imu"
-    gps_sub_topic="/gps"
     mag_sub_topic="/mag"
     baro_sub_topic="/baro"

Commit message: models: add iris_dual_gps model; gazebo_gps_plugin: fix model loading conflict

File: models/rotors_description/urdf/component_snippets.xacro (robot description, xacro)
@@ -59,7 +59,7 @@
         </link>
       </model>
-      <joint name="gps_joint" type="fixed">
+      <joint name="${gps_name}_joint" type="fixed">
         <parent>${parent_link}</parent>
-        <child>gps::link</child>
+        <child>${gps_name}::link</child>
       </joint>
     </gazebo>

File: models/rotors_description/urdf/iris_base.xacro (robot description, xacro)
@@ -78,6 +78,6 @@
   <!-- Mount a GPS module. -->
   <xacro:gps_macro
-    gps_name="gps"
-    pos_x="0.015"
+    gps_name="gps0"
+    pos_x="0.0"
     pos_y="0.0"
     pos_z="0.0"

Commit message: separate the groundtruth into its own model plugin and update the overall model plugins

File: models/rotors_description/urdf/component_snippets.xacro (robot description, xacro)
@@ -171,4 +171,12 @@
         <imuSubTopic>/${imu_sub_topic}</imuSubTopic>
         <motorSpeedCommandPubTopic>/gazebo/command/motor_speed</motorSpeedCommandPubTopic>
+      </plugin>
+    </gazebo>
+  </xacro:macro>
+  <!-- Macro to add the groundtruth_plugin. -->
+  <xacro:macro name="groundtruth_plugin_macro" params="namespace">
+    <gazebo>
+      <plugin name='groundtruth_plugin' filename='libgazebo_groundtruth_plugin.so'>
+        <robotNamespace>${namespace}</robotNamespace>
       </plugin>
     </gazebo>

File: models/rotors_description/urdf/iris_base.xacro (robot description, xacro)
@@ -92,4 +92,9 @@
     parent_link="base_link">
   </xacro:gps_macro>
+  <!-- Instantiate groundtruth plugin. -->
+  <xacro:groundtruth_plugin_macro
+    namespace="${namespace}"
+    >
+  </xacro:groundtruth_plugin_macro>
   <!-- Instantiate magnetometer plugin. -->
   <xacro:magnetometer_plugin_macro

File: models/rotors_description/urdf/plane_base.xacro (robot description, xacro)
@@ -92,4 +92,9 @@
     parent_link="base_link">
   </xacro:gps_macro>
+  <!-- Instantiate groundtruth plugin. -->
+  <xacro:groundtruth_plugin_macro
+    namespace="${namespace}"
+    >
+  </xacro:groundtruth_plugin_macro>
   <!-- Instantiate magnetometer plugin. -->
   <xacro:magnetometer_plugin_macro

File: models/rotors_description/urdf/standard_vtol_base.xacro (robot description, xacro)
@@ -92,4 +92,9 @@
     parent_link="base_link">
   </xacro:gps_macro>
+  <!-- Instantiate groundtruth plugin. -->
+  <xacro:groundtruth_plugin_macro
+    namespace="${namespace}"
+    >
+  </xacro:groundtruth_plugin_macro>
   <!-- Instantiate magnetometer plugin. -->
   <xacro:magnetometer_plugin_macro
