Commit message: Fix inertial sensor oscillation

File: models/rotors_description/urdf/multirotor_base.xacro (robot description, xacro)
@@ -55,4 +55,19 @@
       </plugin>
     </gazebo>
+    <gazebo reference="base_link">
+      <collision name='base_link_inertia_collision'>
+        <surface>
+          <contact>
+            <ode>
+              <min_depth>0.001</min_depth>
+              <max_vel>0.0</max_vel>
+            </ode>
+          </contact>
+          <friction>
+            <ode/>
+          </friction>
+        </surface>
+      </collision>
+   </gazebo>
     <gazebo reference="base_link">
       <material>Gazebo/${color}</material>

Commit message: Merge base link reference tag

File: models/rotors_description/urdf/multirotor_base.xacro (robot description, xacro)
@@ -56,4 +56,5 @@
     </gazebo>
     <gazebo reference="base_link">
+      <material>Gazebo/${color}</material>
       <collision name='base_link_inertia_collision'>
         <surface>
@@ -70,7 +71,4 @@
       </collision>
    </gazebo>
-    <gazebo reference="base_link">
-      <material>Gazebo/${color}</material>
-    </gazebo>
   </xacro:macro>
   <!-- Rotor joint and link -->

Commit message: stabilize plane and standard_vtol contacts

File: models/rotors_description/urdf/multirotor_base.xacro (robot description, xacro)
@@ -54,4 +54,19 @@
         <rotorVelocitySlowdownSim>${rotor_velocity_slowdown_sim}</rotorVelocitySlowdownSim>
       </plugin>
+    </gazebo>
+    <gazebo reference="base_link">
+      <collision name='base_link_inertia_collision'>
+        <surface>
+          <contact>
+            <ode>
+              <min_depth>0.001</min_depth>
+              <max_vel>0.0</max_vel>
+            </ode>
+          </contact>
+          <friction>
+            <ode/>
+          </friction>
+        </surface>
+      </collision>
     </gazebo>
     <gazebo reference="base_link">

Commit message: Fixed color in URDF iris

File: models/rotors_description/urdf/multirotor_base.xacro (robot description, xacro)
@@ -39,4 +39,7 @@
           <!-- <box size="${body_width} ${body_width} ${body_height}"/> --> <!-- [m] [m] [m] -->
         </geometry>
+        <material name="Gazebo/${color}">
+          <color rgba="0. 0. 0. 1"/>
+        </material>
       </visual>
       <collision>
@@ -47,4 +50,7 @@
       </collision>
     </link>
+    <gazebo reference="${robot_namespace}_base_link_inertia">
+      <material>Gazebo/${color}</material>
+    </gazebo>
     <!-- attach multirotor_base_plugin to the base_link -->
     <gazebo>

Commit message: Move meshfiles out of rotors_description
This commit moves the meshfiles out of rotors_description so that we can deprecate rotors_description once the mutlivehicle scripts are based on jinja templates

File: models/rotors_description/urdf/multirotor_base.xacro (robot description, xacro)
@@ -35,5 +35,5 @@
         <origin xyz="0 0 0" rpy="0 0 0" />
         <geometry>
-          <mesh filename="package://rotors_description/meshes/${mesh_file}"
+          <mesh filename="model://iris/meshes/${mesh_file}"
             scale="${mesh_scale}" />
           <!-- <box size="${body_width} ${body_width} ${body_height}"/> --> <!-- [m] [m] [m] -->
@@ -95,5 +95,5 @@
           <!-- <cylinder length="0.005" radius="${radius_rotor}"/> --> <!-- [m] -->
           <!-- <mesh filename="package://rotors_description/meshes/propeller_${direction}.dae" -->
-          <mesh filename="package://rotors_description/meshes/${mesh}_${direction}.dae"
+          <mesh filename="model://iris/meshes/${mesh}_${direction}.dae"
             scale="${mesh_scale}" />
           <!-- <box size="${2*radius_rotor} 0.01 0.005"/> -->
